File: Nanopilot.sch (KiCad schematic (older format))
At the start: 76 parts

Commit message: finalize pin assingment & pullup/down
Parts:
- removed 300k?: R, symbol Device:R
- removed C?: 0.1uF, symbol Device:C_Small
- removed C?: 100nF, symbol Device:C_Small
- removed R? (x2): R_Small, symbol Device:R_Small
- added C?: 100nF, symbol Device:C_Small
- added C? (x2): DNP, symbol Device:C_Small
- added C?: 10nF, symbol Device:C_Small
- added D?: HEARTBEAT, symbol Device:LED
- added J?: ARM, symbol Nanopilot-rescue:Conn_01x04
- added J?: DBG, symbol Connector_Generic:Conn_01x09
- added R? (x8): 10k, symbol Device:R_Small
- added R?: 1k, symbol Device:R_Small
- added R? (x2): 100, symbol Device:R
- added R? (x2): 0, symbol Device:R_Small
- added R?: 220k, symbol Device:R_Small
- added R?: 100k, symbol Device:R_Small
- C?: value C_Small -> 10nF
- R?: renamed from 1.5k; value R -> 1.5k
- R?: renamed from 1.5k?; value R -> 1.5k
- R?: renamed from 3.7k; value R -> 3.7k
- R?: value R_Small -> 220k
- R?: value R_Small -> 100k
- Y?: value Crystal -> 8MHz
Connections:
- net labels added: ARM_LED, ARM_SWITCH, HEARTBEAT_LED, I_bat_sens, NPI_DBG_RX, NPI_DBG_TX, SPEAKER, STM_DBG_RX, STM_DBG_TX, V_bat_sens
- net labels removed: NANOPI_UART1_CTS, NANOPI_UART1_RTS, NANOPI_UART1_RX, NANOPI_UART1_TX
- wire segments 451 -> 527
Other:
- note added: "1.5 A limit\n"
- note added: "230Hz"
- note added: "ADC2_IN1"
- note added: "ADC2_IN2"
- note added: "ADC2_IN3"
- note added: "ADC2_IN4"
- note added: "UART1 RX"
- note added: "UART1 TX"
- note added: "UART3 RX"
- note added: "UART3 TX"
- note added: "UART4 RX"
- note added: "UART4 TX"
- note added: "UART5 RX"
- note removed: "1.517 A limit\n"
