File: sensors.sch (KiCad schematic (older format))
At the start: 24 parts

Commit message: finalize pin assingment & pullup/down
Parts:
- removed L?: L, Inductors_SMD:L_0603, symbol Device:L
- removed R? (x3): 4.7k, symbol Device:R_Small
- added R? (x2): 10k, symbol Device:R_Small
- C?: value 0.1uF -> 100nF
Connections:
- net labels removed: +3.3V, VDDIO
- wire segments 168 -> 176
Other:
- moved on the sheet: U?
