File: airdata/airdata.sch (KiCad schematic (older format))
At the start: 19 parts, among them J1 I2C, J2 I2C, U1 SDP32, U2 MS5611-01BA03, U3 SDP32, U4 LT1761-3.3, U5 HSCMRRN001PD2A3, U6 SDP32

Commit message: airdata footprints & 3d models
Parts:
- C1, C2, C3, C4, C5, C6, C7, C8: footprint (none) -> Capacitor_SMD:C_0603_1608Metric
- J1, J2: footprint (none) -> Connector_JST:JST_GH_BM04B-GHS-TBT_1x04-1MP_P1.25mm_Vertical
- R1, R2, R3: footprint (none) -> Resistor_SMD:R_0603_1608Metric
- U2: footprint (none) -> footprints:MS5611-01BA
- U5: footprint (none) -> footprints:HSCMRRN001PD2A3-side-mount
Changed lines of the file:
@@
 F 0 "J1" H 2880 1342 50  0000 L CNN
 F 1 "I2C" H 2880 1251 50  0000 L CNN
-F 2 "" H 2800 1350 50  0001 C CNN
+F 2 "Connector_JST:JST_GH_BM04B-GHS-TBT_1x04-1MP_P1.25mm_Vertical" H 2800 1350 50  0001 C CNN
 F 3 "~" H 2800 1350 50  0001 C CNN
 	1    2800 1350
@@
 F 0 "J2" H 3680 1342 50  0000 L CNN
 F 1 "I2C" H 3680 1251 50  0000 L CNN
-F 2 "" H 3600 1350 50  0001 C CNN
+F 2 "Connector_JST:JST_GH_BM04B-GHS-TBT_1x04-1MP_P1.25mm_Vertical" H 3600 1350 50  0001 C CNN
 F 3 "~" H 3600 1350 50  0001 C CNN
 	1    3600 1350
@@
 F 0 "C4" H 4542 1546 50  0000 L CNN
 F 1 "1uF" H 4542 1455 50  0000 L CNN
-F 2 "" H 4450 1500 50  0001 C CNN
+F 2 "Capacitor_SMD:C_0603_1608Metric" H 4450 1500 50  0001 C CNN
 F 3 "~" H 4450 1500 50  0001 C CNN
 	1    4450 1500
@@
 F 0 "C6" H 5942 1546 50  0000 L CNN
 F 1 "0.01uF" H 5942 1455 50  0000 L CNN
-F 2 "" H 5850 1500 50  0001 C CNN
+F 2 "Capacitor_SMD:C_0603_1608Metric" H 5850 1500 50  0001 C CNN
 F 3 "~" H 5850 1500 50  0001 C CNN
 	1    5850 1500
@@
 F 0 "C8" H 6392 1546 50  0000 L CNN
 F 1 "10uF" H 6392 1455 50  0000 L CNN
-F 2 "" H 6300 1500 50  0001 C CNN
+F 2 "Capacitor_SMD:C_0603_1608Metric" H 6300 1500 50  0001 C CNN
 F 3 "~" H 6300 1500 50  0001 C CNN
 	1    6300 1500
@@
 F 0 "R1" H 3659 4046 50  0000 L CNN
 F 1 "0" H 3659 3955 50  0000 L CNN
-F 2 "" H 3600 4000 50  0001 C CNN
+F 2 "Resistor_SMD:R_0603_1608Metric" H 3600 4000 50  0001 C CNN
 F 3 "~" H 3600 4000 50  0001 C CNN
 	1    3600 4000
@@
 F 0 "R2" H 5759 4046 50  0000 L CNN
 F 1 "1.2k" H 5759 3955 50  0000 L CNN
-F 2 "" H 5700 4000 50  0001 C CNN
+F 2 "Resistor_SMD:R_0603_1608Metric" H 5700 4000 50  0001 C CNN
 F 3 "~" H 5700 4000 50  0001 C CNN
 	1    5700 4000
@@
 F 0 "R3" H 7759 4046 50  0000 L CNN
 F 1 "2.7k" H 7759 3955 50  0000 L CNN
-F 2 "" H 7700 4000 50  0001 C CNN
+F 2 "Resistor_SMD:R_0603_1608Metric" H 7700 4000 50  0001 C CNN
 F 3 "~" H 7700 4000 50  0001 C CNN
 	1    7700 4000
@@
 F 0 "U2" H 3150 6625 50  0000 C CNN
 F 1 "MS5611-01BA03" H 3150 6534 50  0000 C CNN
-F 2 "" H 3050 6200 50  0001 C CNN
+F 2 "footprints:MS5611-01BA" H 3050 6200 50  0001 C CNN
 F 3 "" H 3050 6200 50  0001 C CNN
 	1    3050 6200
@@
 F 0 "C1" H 2242 3296 50  0000 L CNN
 F 1 "100nF" H 2242 3205 50  0000 L CNN
-F 2 "" H 2150 3250 50  0001 C CNN
+F 2 "Capacitor_SMD:C_0603_1608Metric" H 2150 3250 50  0001 C CNN
 F 3 "~" H 2150 3250 50  0001 C CNN
 	1    2150 3250
@@
 F 0 "C3" H 4342 3296 50  0000 L CNN
 F 1 "100nF" H 4342 3205 50  0000 L CNN
-F 2 "" H 4250 3250 50  0001 C CNN
+F 2 "Capacitor_SMD:C_0603_1608Metric" H 4250 3250 50  0001 C CNN
 F 3 "~" H 4250 3250 50  0001 C CNN
 	1    4250 3250
@@
 F 0 "C7" H 6342 3296 50  0000 L CNN
 F 1 "100nF" H 6342 3205 50  0000 L CNN
-F 2 "" H 6250 3250 50  0001 C CNN
+F 2 "Capacitor_SMD:C_0603_1608Metric" H 6250 3250 50  0001 C CNN
 F 3 "~" H 6250 3250 50  0001 C CNN
 	1    6250 3250
@@
 F 0 "C2" H 2242 6146 50  0000 L CNN
 F 1 "100nF" H 2242 6055 50  0000 L CNN
-F 2 "" H 2150 6100 50  0001 C CNN
+F 2 "Capacitor_SMD:C_0603_1608Metric" H 2150 6100 50  0001 C CNN
 F 3 "~" H 2150 6100 50  0001 C CNN
 	1    2150 6100
@@
 F 0 "C5" H 4742 6246 50  0000 L CNN
 F 1 "100nF" H 4742 6155 50  0000 L CNN
-F 2 "" H 4650 6200 50  0001 C CNN
+F 2 "Capacitor_SMD:C_0603_1608Metric" H 4650 6200 50  0001 C CNN
 F 3 "~" H 4650 6200 50  0001 C CNN
 	1    4650 6200
@@
 F 0 "U5" H 5600 6615 50  0000 C CNN
 F 1 "HSCMRRN001PD2A3" H 5600 6524 50  0000 C CNN
-F 2 "" H 5600 6200 50  0001 C CNN
+F 2 "footprints:HSCMRRN001PD2A3-side-mount" H 5600 6200 50  0001 C CNN
 F 3 "" H 5600 6200 50  0001 C CNN
 	1    5600 6200

Commit message: airdata & power supply pcb
Other:
- note added: "SDP32 (125Pa) up to 50km/h\nSDP31 (500Pa) up to 100km/h\nSDP33 (1500Pa) up to 180km/h"
- note added: "up to 380km/h (6890Pa)"
- note removed: "up to 380km/h"
- note removed: "up to 50km/h"
Changed lines of the file:
@@
 Text Notes 5050 2600 0    50   ~ 0
 beta
-Text Notes 6900 2550 0    50   ~ 0
+Text Notes 6900 2650 0    50   ~ 0
 dynamic pressure
 Text Notes 2850 5550 0    50   ~ 0
 static pressure
-Text Notes 6950 2650 0    50   ~ 0
-up to 50km/h
 Text Notes 5200 5450 0    50   ~ 0
 dynamic pressure
-Text Notes 5250 5550 0    50   ~ 0
-up to 380km/h
+Text Notes 5100 5550 0    50   ~ 0
+up to 380km/h (6890Pa)
 $Comp
 L Device:C_Small C5
@@
 Text Notes 5250 6550 0    50   ~ 0
 I2C Address 0x28
+Text Notes 8950 3250 0    50   ~ 0
+SDP32 (125Pa) up to 50km/h\nSDP31 (500Pa) up to 100km/h\nSDP33 (1500Pa) up to 180km/h
 $EndSCHEMATC
