File: nanopilot/Nanopilot.kicad_pcb (KiCad board)
At the start: 2 copper layers, 19 parts, among them J1 Conn_01x06, J10 Conn_01x06, J11 Conn_01x06, J2 TELEM, J3 GPS, U1 LTC4419, U10 SiP32414, U11 SN74LVC1G08, U12 SN74LVC1G38, U2 NanoPi_Air_1.1, U3 TPS25200, U4 LT1963EST-3.3, U5 LT1761-3.3, U6 TPS25200, U7 STM32F303VETx, U8 SiP32414, U9 SiP32414

Commit message: clean up libraries
Parts:
- U2: footprint symbols_autopilot:NanoPi_Header -> footprints:NanoPi_Header
- moved U2 2.17 mm to (148.0, -156.5)
Connections:
- D2 pad 1: (no net) -> Net-(D2-Pad1)
- J1 pad 3: (no net) -> /I_bat_sens
- J1 pad 4: (no net) -> /V_bat_sens
- U1 pad 11: (no net) -> Net-(U1-Pad11)
- U1 pad 2: (no net) -> Net-(U1-Pad2)
- U1 pad 3: (no net) -> Net-(R2-Pad2)
- U1 pad 4: (no net) -> Net-(R1-Pad2)
- U1 pad 6: (no net) -> Net-(R11-Pad2)
- U1 pad 7: (no net) -> Net-(U1-Pad7)
- U1 pad 8: (no net) -> Net-(U1-Pad8)
- U2 pad A10: (no net) -> /SPEAKER
- U2 pad A11: (no net) -> Net-(U2-PadA11)
- U2 pad A12: (no net) -> Net-(U2-PadA12)
- U2 pad A13: (no net) -> Net-(U2-PadA13)
- U2 pad A14: (no net) -> Net-(U2-PadA14)
- U2 pad A15: (no net) -> Net-(U2-PadA15)
- U2 pad A16: (no net) -> Net-(U2-PadA16)
- U2 pad A17: (no net) -> Net-(U2-PadA17)
- U2 pad A18: (no net) -> /NPI_DBG_RX
- U2 pad A19: (no net) -> Net-(U2-PadA19)
- U2 pad A20: (no net) -> /NPI_DBG_TX
- U2 pad A21: (no net) -> Net-(U2-PadA21)
- U2 pad A3: (no net) -> /USB2_D+
- U2 pad A5: (no net) -> /USB2_D-
- U2 pad A7: (no net) -> /USB3_D+
- U2 pad A9: (no net) -> /USB3_D-
- U2 pad B19: (no net) -> Net-(U2-PadB19)
- U2 pad B21: (no net) -> Net-(U2-PadB21)
- U2 pad B23: (no net) -> Net-(U2-PadB23)
- U2 pad B24: (no net) -> Net-(U2-PadB24)
- U2 pad B3: (no net) -> /NANOPI_I2C_SDA
- U2 pad B5: (no net) -> /NANOPI_I2C_SCL
- U3 pad 2: (no net) -> Net-(R12-Pad1)
- U3 pad 3: (no net) -> Net-(R13-Pad2)
- U3 pad 4: (no net) -> Net-(R8-Pad1)
- U5 pad 4: (no net) -> Net-(C13-Pad2)
- U5 pad 5: (no net) -> /3V3_SENS
- U6 pad 2: (no net) -> Net-(R18-Pad1)
- U6 pad 3: (no net) -> Net-(R19-Pad2)
- U7 pad 10: (no net) -> Net-(U7-Pad10)
- U7 pad 11: (no net) -> Net-(U7-Pad11)
- U7 pad 12: (no net) -> Net-(C16-Pad1)
- U7 pad 13: (no net) -> Net-(C17-Pad1)
- U7 pad 15: (no net) -> /SERVO1_PWM
- U7 pad 16: (no net) -> /SERVO2_PWM
- U7 pad 17: (no net) -> /SERVO3_PWM
- U7 pad 18: (no net) -> /SERVO4_PWM
- U7 pad 19: (no net) -> Net-(U7-Pad19)
- U7 pad 29: (no net) -> /5V_IN_ADC
- U7 pad 30: (no net) -> /V_SERVO_ADC
- U7 pad 31: (no net) -> /I_bat_adc
- U7 pad 32: (no net) -> /V_bat_adc
- U7 pad 33: (no net) -> /STM_DBG_TX
- U7 pad 34: (no net) -> /STM_DBG_RX
- U7 pad 37: (no net) -> Net-(U7-Pad37)
- U7 pad 39: (no net) -> /HEARTBEAT_LED
- U7 pad 40: (no net) -> /ARM_LED
- U7 pad 41: (no net) -> /ARM_SWITCH
- U7 pad 42: (no net) -> Net-(U7-Pad42)
- U7 pad 43: (no net) -> Net-(U7-Pad43)
- U7 pad 44: (no net) -> Net-(U7-Pad44)
- U7 pad 45: (no net) -> Net-(U7-Pad45)
- U7 pad 46: (no net) -> Net-(U7-Pad46)
- U7 pad 47: (no net) -> Net-(R22-Pad1)
- U7 pad 48: (no net) -> /RSSI/TELEM
- U7 pad 51: (no net) -> Net-(U7-Pad51)
- U7 pad 52: (no net) -> /SPI_SENS_SCLK
- U7 pad 53: (no net) -> /SPI_SENS_MISO
- U7 pad 54: (no net) -> /SPI_SENS_MOSI
- U7 pad 55: (no net) -> Net-(U7-Pad55)
- U7 pad 56: (no net) -> Net-(U7-Pad56)
- U7 pad 57: (no net) -> /~LSM_CS
- U7 pad 58: (no net) -> /~MPU_CS
- U7 pad 59: (no net) -> /H3LIS_INT
- U7 pad 60: (no net) -> /LIS3MDL_INT
- U7 pad 61: (no net) -> /MPU_INT
- U7 pad 62: (no net) -> /LSM_INT1
- U7 pad 63: (no net) -> /SERVO5_PWM
- U7 pad 64: (no net) -> /SERVO6_PWM
- U7 pad 65: (no net) -> /SERVO7_PWM
- U7 pad 66: (no net) -> /SERVO8_PWM
- U7 pad 67: (no net) -> Net-(U7-Pad67)
- U7 pad 7: (no net) -> Net-(U7-Pad7)
- U7 pad 72: (no net) -> /SWDIO
- U7 pad 73: (no net) -> Net-(U7-Pad73)
- U7 pad 76: (no net) -> /SWCLK
- U7 pad 77: (no net) -> Net-(U7-Pad77)
- U7 pad 8: (no net) -> Net-(U7-Pad8)
- U7 pad 80: (no net) -> Net-(U7-Pad80)
- U7 pad 81: (no net) -> Net-(U7-Pad81)
- U7 pad 82: (no net) -> Net-(U7-Pad82)
- U7 pad 83: (no net) -> Net-(R21-Pad2)
- U7 pad 84: (no net) -> Net-(U7-Pad84)
- U7 pad 85: (no net) -> Net-(U7-Pad85)
- U7 pad 86: (no net) -> Net-(U7-Pad86)
- U7 pad 87: (no net) -> Net-(U7-Pad87)
- U7 pad 88: (no net) -> Net-(U7-Pad88)
- U7 pad 89: (no net) -> Net-(U7-Pad89)
- U7 pad 9: (no net) -> Net-(U7-Pad9)
- U7 pad 92: (no net) -> /I2C_SENS_SCL
- U7 pad 93: (no net) -> /I2C_SENS_SDA
- U8 pad 5: (no net) -> /I2C_POWER
- U9 pad 5: (no net) -> /USB3_POWER
- U9 pad 8: (no net) -> /USB2_POWER

Commit message: version ready to be routed
Parts:
- added C1: 10nF, Capacitor_SMD:C_0603_1608Metric, B.Cu at (90.8, 32.0)
- added C10: DNP, Capacitor_SMD:C_0603_1608Metric, B.Cu at (97.5, 33.8)
- added C11: DNP, Capacitor_SMD:C_0603_1608Metric, B.Cu at (100.5, 33.6)
- added C12: 10uF, Capacitor_SMD:C_0603_1608Metric, B.Cu at (114.2, 57.8)
- added C13: 0.01uF, Capacitor_SMD:C_0603_1608Metric, F.Cu at (106.7, 46.0)
- added C14: 10uF, Capacitor_SMD:C_0603_1608Metric, F.Cu at (106.7, 44.4)
- added C15: 22uF, Capacitor_SMD:C_0805_2012Metric, B.Cu at (113.8, 38.2)
- added C16: 22pF, Capacitor_SMD:C_0603_1608Metric, B.Cu at (88.8, 50.0)
- added C17: 22pF, Capacitor_SMD:C_0603_1608Metric, B.Cu at (87.8, 42.5)
- added C18: 100nF, Capacitor_SMD:C_0603_1608Metric, B.Cu at (86.5, 52.2)
- added C19: 100nF, Capacitor_SMD:C_0603_1608Metric, B.Cu at (94.5, 35.2)
- added C20: 100nF, Capacitor_SMD:C_0603_1608Metric, B.Cu at (108.2, 36.2)
- added C21: 100nF, Capacitor_SMD:C_0603_1608Metric, B.Cu at (94.8, 55.0)
- added C22: 100nF, Capacitor_SMD:C_0603_1608Metric, B.Cu at (110.0, 50.5)
- added C23: 100nF, Capacitor_SMD:C_0603_1608Metric, B.Cu at (89.8, 40.5)
- added C24: 47uF, Capacitor_SMD:C_1206_3216Metric, B.Cu at (125.8, 41.0)
- added C25: 47uF, Capacitor_SMD:C_1206_3216Metric, B.Cu at (76.8, 32.2)
- added C26: 47uF, Capacitor_SMD:C_1206_3216Metric, B.Cu at (74.8, 49.8)
- added C27: 47uF, Capacitor_SMD:C_1206_3216Metric, B.Cu at (126.8, 58.5)
- added C28: 0.1uF, Capacitor_SMD:C_0603_1608Metric, B.Cu at (123.0, 59.2)
- added C29: 0.1uF, Capacitor_SMD:C_0603_1608Metric, B.Cu at (73.2, 31.8)
- added C3: 10nF, Capacitor_SMD:C_0603_1608Metric, B.Cu at (87.9, 32.0)
- added C30: 0.1uF, Capacitor_SMD:C_0603_1608Metric, B.Cu at (121.7, 39.5)
- added C31: 0.1uF, Capacitor_SMD:C_0603_1608Metric, B.Cu at (120.5, 58.0)
- added C32: 0.1uF, Capacitor_SMD:C_0603_1608Metric, F.Cu at (96.2, 37.5)
- added C33: 0.1uF, Capacitor_SMD:C_0603_1608Metric, B.Cu at (121.7, 38.0)
- added C34: 100nF, Capacitor_SMD:C_0603_1608Metric, B.Cu at (97.5, 58.2)
- added C35: 100nF, Capacitor_SMD:C_0603_1608Metric, F.Cu at (89.2, 42.5)
- added C36: 10nF, Capacitor_SMD:C_0603_1608Metric, F.Cu at (103.5, 47.6)
- added C37: 0.1uF, Capacitor_SMD:C_0603_1608Metric, F.Cu at (94.2, 40.8)
- added C38: 100nF, Capacitor_SMD:C_0603_1608Metric, F.Cu at (100.2, 48.0)
- added C39: 1uF, Capacitor_SMD:C_0603_1608Metric, B.Cu at (121.7, 41.0)
- added C4: 22uF, Capacitor_SMD:C_0805_2012Metric, F.Cu at (111.2, 56.5)
- added C40: 0.1uF, Capacitor_SMD:C_0603_1608Metric, F.Cu at (96.5, 42.9)
- added C41: 0.1uF, Capacitor_SMD:C_0603_1608Metric, F.Cu at (103.5, 44.5)
- added C42: 10uF, Capacitor_SMD:C_0603_1608Metric, F.Cu at (97.3, 51.0)
- added C43: 1uF, Capacitor_SMD:C_0603_1608Metric, F.Cu at (92.5, 47.8)
- added C44: 1uF, Capacitor_SMD:C_0603_1608Metric, F.Cu at (95.8, 47.8)
- added C45: 0.1uF, Capacitor_SMD:C_0603_1608Metric, F.Cu at (103.5, 50.9)
- added C46: 100nF, Capacitor_SMD:C_0603_1608Metric, F.Cu at (92.7, 43.4)
- added C47: 100nF, Capacitor_SMD:C_0603_1608Metric, F.Cu at (99.2, 37.6)
- added C5: 22uF, Capacitor_SMD:C_0805_2012Metric, F.Cu at (111.2, 54.5)
- added C6: 1uF, Capacitor_SMD:C_0603_1608Metric, F.Cu at (106.7, 52.4)
- added C7: 10uF, Capacitor_SMD:C_0603_1608Metric, B.Cu at (114.2, 54.8)
- added C8: 22uF, Capacitor_SMD:C_0805_2012Metric, F.Cu at (110.0, 40.0)
- added C9: 100uF, Capacitor_SMD:C_0805_2012Metric, B.Cu at (113.8, 45.2)
- added D1: 5V UV, LED_SMD:LED_0603_1608Metric, B.Cu at (97.5, 30.8)
- added D3: OC PERIPHERAL, LED_SMD:LED_0603_1608Metric, B.Cu at (103.7, 30.8)
- added D4: HEARTBEAT, LED_SMD:LED_0603_1608Metric, B.Cu at (100.5, 30.8)
- added J12: Servo Right, footprints:pin_headers_smd_2x03_P2.54mm_horizontal, F.Cu at (125.5, 48.5)
- added J13: Servo Right, footprints:pin_headers_smd_2x03_P2.54mm_horizontal, F.Cu at (125.5, 41.5)
- added J14: Servo Left, footprints:pin_headers_smd_2x03_P2.54mm_horizontal, F.Cu at (75.0, 48.5)
- added J15: Servo Left, footprints:pin_headers_smd_2x03_P2.54mm_horizontal, F.Cu at (75.0, 41.5)
- added J16: servo left, Connector_Molex:Molex_Pico-Lock_504050-0691_1x06-1MP_P1.50mm_Horizontal, B.Cu at (68.8, 52.5)
- added J17: servo right, Connector_Molex:Molex_Pico-Lock_504050-0691_1x06-1MP_P1.50mm_Horizontal, B.Cu at (131.8, 52.5)
- added J4: USB1, Connector_JST:JST_GH_SM04B-GHS-TB_1x04-1MP_P1.25mm_Horizontal, F.Cu at (132.2, 34.5)
- added J5: USB2, Connector_JST:JST_GH_SM04B-GHS-TB_1x04-1MP_P1.25mm_Horizontal, F.Cu at (132.2, 43.8)
- added J6: I2C, Connector_JST:JST_GH_SM04B-GHS-TB_1x04-1MP_P1.25mm_Horizontal, F.Cu at (68.5, 34.6)
- added J7: ARM, Connector_JST:JST_GH_SM05B-GHS-TB_1x05-1MP_P1.25mm_Horizontal, F.Cu at (68.5, 44.4)
- added J8: DBG, Connector_Molex:Molex_PicoBlade_53261-0971_1x09-1MP_P1.25mm_Horizontal, F.Cu at (100.2, 56.8)
- added J9: RX, Connector_JST:JST_GH_SM05B-GHS-TB_1x05-1MP_P1.25mm_Horizontal, F.Cu at (68.5, 54.9)
- added L1: L_Small, Inductor_SMD:L_0603_1608Metric, B.Cu at (89.8, 37.8)
- added MH1: MountingHole_Pad, MountingHole:MountingHole_2.2mm_M2_Pad_Via, F.Cu at (67.8, 27.5)
- added MH2: MountingHole_Pad, MountingHole:MountingHole_2.2mm_M2_Pad_Via, F.Cu at (67.8, 62.5)
- added MH3: MountingHole_Pad, MountingHole:MountingHole_2.2mm_M2_Pad_Via, F.Cu at (132.8, 27.5)
- added MH4: MountingHole_Pad, MountingHole:MountingHole_2.2mm_M2_Pad_Via, F.Cu at (132.8, 62.5)
- added R1: 812k, Resistor_SMD:R_0603_1608Metric, F.Cu at (111.1, 44.0)
- added R10: 100k, Resistor_SMD:R_0603_1608Metric, B.Cu at (87.9, 30.8)
- added R11: 3.7k, Resistor_SMD:R_0603_1608Metric, F.Cu at (109.3, 45.7)
- added R12: 33k 1%, Resistor_SMD:R_0603_1608Metric, F.Cu at (108.2, 39.8)
- added R13: 1.5k, Resistor_SMD:R_0603_1608Metric, F.Cu at (107.9, 42.8)
- added R14: 0, Resistor_SMD:R_0603_1608Metric, B.Cu at (97.5, 35.2)
- added R15: 0, Resistor_SMD:R_0603_1608Metric, B.Cu at (100.5, 35.0)
- added R16: 4.7k, Resistor_SMD:R_0603_1608Metric, B.Cu at (85.5, 32.5)
- added R17: 4.7k, Resistor_SMD:R_0603_1608Metric, B.Cu at (86.7, 36.1)
- added R18: 64k 1%, Resistor_SMD:R_0603_1608Metric, B.Cu at (114.0, 40.2)
- added R19: 1.5k, Resistor_SMD:R_0603_1608Metric, B.Cu at (112.2, 31.5)
- added R2: 247k, Resistor_SMD:R_0603_1608Metric, F.Cu at (111.8, 46.5)
- added R20: 100k, Resistor_SMD:R_0603_1608Metric, B.Cu at (86.5, 55.2)
- added R21: 100, Resistor_SMD:R_0603_1608Metric, B.Cu at (102.8, 55.5)
- added R22: 100, Resistor_SMD:R_0603_1608Metric, B.Cu at (105.8, 34.2)
- added R23: 1k, Resistor_SMD:R_0603_1608Metric, B.Cu at (100.5, 32.2)
- added R24: 10k, Resistor_SMD:R_0603_1608Metric, B.Cu at (122.5, 54.0)
- added R25: 10k, Resistor_SMD:R_0603_1608Metric, B.Cu at (122.3, 32.6)
- added R26: 10k, Resistor_SMD:R_0603_1608Metric, F.Cu at (89.8, 48.5)
- added R27: 10k, Resistor_SMD:R_0603_1608Metric, B.Cu at (121.0, 54.0)
- added R28: 10k, Resistor_SMD:R_0603_1608Metric, B.Cu at (120.8, 32.6)
- added R29: 10k, Resistor_SMD:R_0603_1608Metric, F.Cu at (88.2, 48.5)
- added R3: 100k, Resistor_SMD:R_0603_1608Metric, F.Cu at (112.6, 44.0)
- added R30: 10k, Resistor_SMD:R_0603_1608Metric, B.Cu at (95.2, 59.0)
- added R31: 10k, Resistor_SMD:R_0603_1608Metric, F.Cu at (89.2, 37.8)
- added R32: 10k, Resistor_SMD:R_0603_1608Metric, B.Cu at (92.2, 57.8)
- added R33: 10k, Resistor_SMD:R_0603_1608Metric, F.Cu at (100.0, 40.6)
- added R34: 10k, Resistor_SMD:R_0603_1608Metric, F.Cu at (97.2, 45.3)
- added R35: 4.7k, Resistor_SMD:R_0603_1608Metric, F.Cu at (89.2, 52.8)
- added R36: 4.7k, Resistor_SMD:R_0603_1608Metric, F.Cu at (89.2, 54.5)
- added R37: 200, Resistor_SMD:R_0603_1608Metric, B.Cu at (126.5, 38.9)
- added R38: 200, Resistor_SMD:R_0603_1608Metric, B.Cu at (126.5, 37.2)
- added R39: 200, Resistor_SMD:R_0603_1608Metric, B.Cu at (74.2, 41.8)
- added R4: 220k, Resistor_SMD:R_0603_1608Metric, B.Cu at (90.8, 33.2)
- added R40: 200, Resistor_SMD:R_0603_1608Metric, B.Cu at (74.2, 43.2)
- added R41: 200, Resistor_SMD:R_0603_1608Metric, B.Cu at (74.5, 36.5)
- added R42: 200, Resistor_SMD:R_0603_1608Metric, B.Cu at (74.5, 38.0)
- added R43: 200, Resistor_SMD:R_0603_1608Metric, B.Cu at (126.3, 32.7)
- added R44: 200, Resistor_SMD:R_0603_1608Metric, B.Cu at (126.5, 30.9)
- added R45: 200, Resistor_SMD:R_0603_1608Metric, B.Cu at (74.0, 51.5)
- added R46: 200, Resistor_SMD:R_0603_1608Metric, B.Cu at (74.0, 53.0)
- added R47: 200, Resistor_SMD:R_0603_1608Metric, B.Cu at (74.3, 56.8)
- added R48: 200, Resistor_SMD:R_0603_1608Metric, B.Cu at (74.3, 58.2)
- added R49: 200, Resistor_SMD:R_0603_1608Metric, B.Cu at (126.2, 53.2)
- added R5: 100k, Resistor_SMD:R_0603_1608Metric, B.Cu at (90.8, 30.8)
- added R50: 200, Resistor_SMD:R_0603_1608Metric, B.Cu at (126.2, 51.8)
- added R51: 200, Resistor_SMD:R_0603_1608Metric, B.Cu at (126.2, 50.2)
- added R52: 200, Resistor_SMD:R_0603_1608Metric, B.Cu at (126.2, 48.8)
- added R6: 4.7k, Resistor_SMD:R_0603_1608Metric, B.Cu at (111.5, 48.5)
- added R7: 4.7k, Resistor_SMD:R_0603_1608Metric, B.Cu at (111.5, 47.0)
- added R8: 300k, Resistor_SMD:R_0603_1608Metric, F.Cu at (103.3, 39.8)
- added R9: 220k, Resistor_SMD:R_0603_1608Metric, B.Cu at (87.9, 33.2)
- added REF**: axes, footprints:axes, B.Cu at (89.8, 59.2)
- added TP1: Time, TestPoint:TestPoint_Pad_D1.0mm, B.Cu at (120.2, 42.5)
- added TP10: MISO, TestPoint:TestPoint_Pad_D1.0mm, B.Cu at (111.2, 39.2)
- added TP11: MOSI, TestPoint:TestPoint_Pad_D1.0mm, B.Cu at (111.5, 41.0)
- added TP12: CTS, TestPoint:TestPoint_Pad_D1.0mm, B.Cu at (80.0, 48.8)
- added TP13: RTS, TestPoint:TestPoint_Pad_D1.0mm, B.Cu at (80.0, 51.2)
- added TP14: TX, TestPoint:TestPoint_Pad_D1.0mm, B.Cu at (80.0, 41.0)
- added TP15: RX, TestPoint:TestPoint_Pad_D1.0mm, B.Cu at (80.0, 38.8)
- added TP16: SCL, TestPoint:TestPoint_Pad_D1.0mm, B.Cu at (99.2, 56.0)
- added TP17: SDA, TestPoint:TestPoint_Pad_D1.0mm, B.Cu at (97.8, 55.5)
- added TP2: CS_LSM, TestPoint:TestPoint_Pad_D1.0mm, B.Cu at (111.8, 42.8)
- added TP3: CS_MPU, TestPoint:TestPoint_Pad_D1.0mm, B.Cu at (110.5, 43.8)
- added TP4: TestPoint, TestPoint:TestPoint_Pad_D1.0mm, B.Cu at (106.2, 31.2)
- added TP5: TestPoint, TestPoint:TestPoint_Pad_D1.0mm, B.Cu at (107.2, 32.0)
- added TP6: TestPoint, TestPoint:TestPoint_Pad_D1.0mm, B.Cu at (108.2, 31.2)
- added TP7: TestPoint, TestPoint:TestPoint_Pad_D1.0mm, B.Cu at (109.2, 32.0)
- added TP8: TestPoint, TestPoint:TestPoint_Pad_D1.0mm, B.Cu at (110.2, 31.2)
- added TP9: SCL, TestPoint:TestPoint_Pad_D1.0mm, B.Cu at (111.0, 37.8)
- added U13: LSM6DSM, footprints:PQFN50P300X250X86-14N, F.Cu at (97.0, 40.3)
- added U14: MPU-9250, footprints:MPU-9250_QFN-24_0.4mm, F.Cu at (100.2, 45.0)
- added U15: 24LC256, Package_SO:SOIC-8_3.9x4.9mm_P1.27mm, B.Cu at (124.5, 45.2)
- added U16: MS5611-01BA03, footprints:MS5611-01BA, F.Cu at (93.8, 51.0)
- added U17: LIS3MDL, footprints:LGA12R50P4X4_200X200X100, F.Cu at (92.5, 45.8)
- added U18: H3LIS331DL, footprints:H3LIS331DL, F.Cu at (100.2, 50.9)
- added Y1: 8MHz, Crystal:Crystal_SMD_Abracon_ABM3C-4Pin_5.0x3.2mm, B.Cu at (88.8, 46.2)
- D2: footprint Diode_SMD:D_0603_1608Metric -> LED_SMD:LED_0603_1608Metric; moved to B.Cu
- J10: value Conn_01x06 -> servo left; moved to B.Cu
- J11: value Conn_01x06 -> servo right; moved to B.Cu
- U12, U4, U7, U8, U9: moved to B.Cu
- U3: footprint symbols_autopilot:TPS25200_WSON_6 -> footprints:TPS25200_WSON_6
- U6: footprint symbols_autopilot:TPS25200_WSON_6 -> footprints:TPS25200_WSON_6; moved to B.Cu
- moved U12 239.8 mm to (95.0, 57.1)
- moved U4 236.1 mm to (109.0, 56.5), turned to 180 degrees
- moved J11 229.2 mm to (68.8, 37.5), turned to 270 degrees
- moved U8 215.8 mm to (122.3, 57.0), turned to 270 degrees
- moved J3 215.6 mm to (132.2, 54.2), turned to 90 degrees
- moved U11 212.5 mm to (89.2, 40.1), turned to 270 degrees
- moved U1 211.0 mm to (110.8, 50.2), turned to 270 degrees
- moved J1 209.1 mm to (105.8, 34.0)
- moved U2 207.1 mm to (100.2, 45.0)
- moved U7 206.3 mm to (100.2, 45.0)
- moved J10 202.3 mm to (131.8, 37.4), turned to 90 degrees
- moved U5 198.3 mm to (106.8, 49.3), turned to 90 degrees
- moved U3 197.9 mm to (106.0, 40.2), turned to 180 degrees
- moved U6 197.3 mm to (113.8, 42.8), turned to 270 degrees
- moved U10 194.0 mm to (89.0, 45.2), turned to 90 degrees
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Connections:
- U1 pad 11: Net-(U1-Pad11) -> (no net)
- U1 pad 2: Net-(U1-Pad2) -> (no net)
- U1 pad 7: Net-(U1-Pad7) -> (no net)
- U1 pad 8: Net-(U1-Pad8) -> (no net)
- U10 pad 3: /GPS_POWER_EN -> /I2C_POWER_EN
- U10 pad 5: /GPS_POWER -> /I2C_POWER
- U2 pad A11: Net-(U2-PadA11) -> /TIME_SYNC
- U7 pad 10: Net-(U7-Pad10) -> (no net)
- U7 pad 11: Net-(U7-Pad11) -> (no net)
- U7 pad 15: /SERVO1_PWM -> Net-(R45-Pad2)
- U7 pad 16: /SERVO2_PWM -> Net-(R46-Pad2)
- U7 pad 17: /SERVO3_PWM -> Net-(R47-Pad2)
- U7 pad 18: /SERVO4_PWM -> Net-(R48-Pad2)
- U7 pad 19: Net-(U7-Pad19) -> (no net)
- U7 pad 35: /SERVO15_PWM -> Net-(R39-Pad2)
- U7 pad 36: /SERVO16_PWM -> Net-(R40-Pad2)
- U7 pad 37: Net-(U7-Pad37) -> (no net)
- U7 pad 51: Net-(U7-Pad51) -> (no net)
- U7 pad 55: Net-(U7-Pad55) -> (no net)
- U7 pad 56: Net-(U7-Pad56) -> /TIME_SYNC
- U7 pad 63: /SERVO5_PWM -> Net-(R49-Pad2)
- U7 pad 64: /SERVO6_PWM -> Net-(R50-Pad2)
- U7 pad 65: /SERVO7_PWM -> Net-(R51-Pad2)
- U7 pad 66: /SERVO8_PWM -> Net-(R52-Pad2)
- U7 pad 67: Net-(U7-Pad67) -> (no net)
- U7 pad 7: Net-(U7-Pad7) -> (no net)
- U7 pad 70: /SERVO9_PWM -> Net-(R37-Pad2)
- U7 pad 71: /SERVO10_PWM -> Net-(R38-Pad2)
- U7 pad 73: Net-(U7-Pad73) -> (no net)
- U7 pad 77: Net-(U7-Pad77) -> (no net)
- U7 pad 8: Net-(U7-Pad8) -> (no net)
- U7 pad 80: Net-(U7-Pad80) -> (no net)
- U7 pad 81: Net-(U7-Pad81) -> (no net)
- U7 pad 82: Net-(U7-Pad82) -> (no net)
- U7 pad 84: Net-(U7-Pad84) -> (no net)
- U7 pad 85: Net-(U7-Pad85) -> (no net)
- U7 pad 86: Net-(U7-Pad86) -> (no net)
- U7 pad 87: Net-(U7-Pad87) -> (no net)
- U7 pad 88: Net-(U7-Pad88) -> (no net)
- U7 pad 89: Net-(U7-Pad89) -> (no net)
- U7 pad 9: Net-(U7-Pad9) -> (no net)
- U7 pad 90: /SERVO13_PWM -> Net-(R41-Pad2)
- U7 pad 91: /SERVO14_PWM -> Net-(R42-Pad2)
- U7 pad 95: /SERVO11_PWM -> Net-(R43-Pad2)
- U7 pad 96: /SERVO12_PWM -> Net-(R44-Pad2)
- U8 pad 3: /I2C_POWER_EN -> /GPS_POWER_EN
- U8 pad 5: /I2C_POWER -> /GPS_POWER
Routing:
- net /V_SERVO: track 0.00 -> 60.2 mm, vias 0 -> 11
- net /TELEM_RX: track 0.00 -> 29.8 mm, vias 0 -> 1
- net /TELEM_CTS: track 0.00 -> 19.6 mm
- net /TELEM_RTS: track 0.00 -> 17.5 mm
- net /NANOPI_I2C_SCL: track 0.00 -> 16.5 mm
- net /TELEM_TX: track 0.00 -> 16.3 mm, vias 0 -> 1
- net /NRST: track 0.00 -> 14.8 mm, vias 0 -> 1
- net /3V3_SENS: track 0.00 -> 13.0 mm
- net /STM_CTRL_BOOTLOADER: track 0.00 -> 9.77 mm, vias 0 -> 1
- net /I_bat_sens: track 0.00 -> 8.88 mm, vias 0 -> 1
- net Net-(C16-Pad1): track 0.00 -> 8.45 mm
- net Net-(C17-Pad1): track 0.00 -> 5.41 mm
- net GND: track 0.00 -> 5.25 mm
- net /LL_CTRL_POWER: track 0.00 -> 5.06 mm
- net /~LSM_CS: track 0.00 -> 3.91 mm
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- added copper zone on In2.Cu, net /V_SERVO
Other:
- board outline added: 70 x 40 mm
- copper layers 2 -> 4
- rule trace_min: 0.2 -> 0.16
- board text added: "+ +"
- board text added: "- -"
- board text added: "1 2"
- board text added: "3 4"
- board text added: "5 6"
- board text added: "5V"
- board text added: "7 8"
- board text added: "ARM"
- board text added: "GPS"
- board text added: "I2C"
- board text added: "OC"
- board text added: "POWER"
- board text added: "Peri"
- board text added: "RX"
- board text added: "S 13…16"
- board text added: "S 1…4"
- board text added: "S 5...8"
- board text added: "S 9…12"
- board text added: "USB"
- board text added: "UV"
