File: nanopilot/Nanopilot.kicad_pcb (KiCad board)
At the start: 4 copper layers, 70 x 40 mm, 162 parts, among them J1 Conn_01x06, J10 servo left, J11 servo right, J12 Servo Right, J13 Servo Right, J14 Servo Left, J15 Servo Left, J16 servo left, J17 servo right, J2 TELEM, J3 GPS, J4 USB1, J5 USB2, J6 I2C, J7 ARM, J8 DBG, J9 RX, U1 LTC4419, U10 SiP32414, U11 SN74LVC1G08, U12 SN74LVC1G38, U13 LSM6DSM, U14 MPU-9250, U15 24LC256, U16 MS5611-01BA03, U17 LIS3MDL, U18 H3LIS331DL, U2 NanoPi_Air_1.1, U3 TPS25200, U4 LT1963EST-3.3, U5 LT1761-3.3, U6 TPS25200, U7 STM32F303VETx, U8 SiP32414, U9 SiP32414, Y1 8MHz

Commit message: routing nanopilot WIP
Parts:
- moved C47 8.66 mm to (96.5, 45.8), turned to 0 degrees
- moved R13 5.68 mm to (112.5, 39.4), turned to 270 degrees
- moved R34 5.52 mm to (101.0, 41.2), turned to 180 degrees
- moved C43 4.70 mm to (92.7, 43.1)
- moved R49 4.55 mm to (126.2, 48.7)
- moved R52 4.45 mm to (126.2, 53.2)
- moved R33 4.24 mm to (97.2, 43.7), turned to 90 degrees
- moved R7 3.24 mm to (112.5, 50.1), turned to 90 degrees
- moved R50 1.65 mm to (126.2, 50.1)
- moved R6 1.62 mm to (111.2, 50.1), turned to 90 degrees
- moved R39 1.51 mm to (74.0, 40.2)
- moved R40 1.51 mm to (74.0, 41.8)
- moved R51 1.45 mm to (126.2, 51.7)
- moved R29 1.30 mm to (88.8, 49.7), turned to 0 degrees
- moved R14 1.25 mm to (97.5, 34.0)
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Connections:
- R49 pad 1: /SERVO5_PWM -> /SERVO8_PWM
- R50 pad 1: /SERVO6_PWM -> /SERVO7_PWM
- R51 pad 1: /SERVO7_PWM -> /SERVO6_PWM
- R52 pad 1: /SERVO8_PWM -> /SERVO5_PWM
- U7 pad 1: /I2C_POWER_EN -> /TELEM_POWER_EN
- U7 pad 3: /USB3_POWER_EN -> /GPS_POWER_EN
- U7 pad 4: /TELEM_POWER_EN -> /I2C_POWER_EN
- U7 pad 5: /GPS_POWER_EN -> /USB3_POWER_EN
- U7 pad 59: /H3LIS_INT -> /MPU_INT
- U7 pad 60: /LIS3MDL_INT -> /LSM_INT1
- U7 pad 61: /MPU_INT -> /H3LIS_INT
- U7 pad 62: /LSM_INT1 -> /LIS3MDL_INT
Routing:
- net Net-(R44-Pad2): track 0.00 -> 75.3 mm, vias 0 -> 2
- net Net-(R43-Pad2): track 0.00 -> 73.2 mm, vias 0 -> 2
- net /SPEAKER: track 0.00 -> 64.7 mm, vias 0 -> 1
- net Net-(R41-Pad2): track 0.00 -> 60.5 mm, vias 0 -> 2
- net /ARM_LED: track 0.00 -> 56.7 mm, vias 0 -> 2
- net Net-(R42-Pad2): track 0.00 -> 54.4 mm, vias 0 -> 2
- net /RSSI/TELEM: track 0.00 -> 53.9 mm, vias 0 -> 2
- net Net-(R38-Pad2): track 0.00 -> 53.3 mm, vias 0 -> 2
- net /ARM_SWITCH: track 0.00 -> 52.7 mm, vias 0 -> 2
- net /USB3_POWER_EN: track 0.00 -> 52.1 mm, vias 0 -> 2
- net Net-(R37-Pad2): track 0.00 -> 52.0 mm, vias 0 -> 2
- net /USB2_POWER_EN: track 0.00 -> 50.9 mm, vias 0 -> 2
- net /RC_IN: track 0.00 -> 36.6 mm, vias 0 -> 1
- net /NANOPI_POWER_EN: track 0.00 -> 35.2 mm
- net /GPS_POWER_EN: track 0.00 -> 33.5 mm
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- added copper zone on In1.Cu, net GND
Other:
- net class Default: clearance 0.2 -> 0.16
- rule trace_clearance: 0.2 -> 0.16
- board text added: "TELEM"

Commit message: routing WIP
Parts:
- C10, R14: moved to F.Cu
- U15: footprint Package_SO:SOIC-8_3.9x4.9mm_P1.27mm -> Package_SO:MSOP-8_3x3mm_P0.65mm
- moved U15 38.8 mm to (86.9, 54.9), turned to 90 degrees
- moved C39 34.4 mm to (90.0, 54.6), turned to 270 degrees
- moved R27 24.8 mm to (96.5, 57.8), turned to 0 degrees
- moved U8 24.0 mm to (122.8, 33.0)
- moved C31 23.5 mm to (121.0, 34.5)
- moved R24 20.1 mm to (114.1, 35.8), turned to 0 degrees
- moved R20 10.7 mm to (96.5, 59.0), turned to 0 degrees
- moved C18 9.86 mm to (95.4, 56.6), turned to 180 degrees
- moved R25 7.54 mm to (114.9, 31.5)
- moved R28 7.34 mm to (113.6, 31.5)
- moved C10 5.15 mm to (98.5, 37.7), turned to 270 degrees
- moved R32 5.09 mm to (87.3, 59.1), turned to 180 degrees
- moved R14 4.55 mm to (100.2, 37.7), turned to 270 degrees
- moved C28 4.47 mm to (126.4, 56.4)
- moved C34 4.00 mm to (93.5, 58.4)
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Connections:
- C30 pad 2: /USB3_POWER -> /USB2_POWER
- C33 pad 2: /USB2_POWER -> /USB3_POWER
- R25 pad 2: /USB3_POWER_EN -> /USB2_POWER_EN
- R28 pad 2: /USB2_POWER_EN -> /USB3_POWER_EN
- U10 pad 2: /TELEM_POWER_EN -> /I2C_POWER_EN
- U10 pad 3: /I2C_POWER_EN -> /TELEM_POWER_EN
- U10 pad 5: /I2C_POWER -> /TELEM_POWER
- U10 pad 8: /TELEM_POWER -> /I2C_POWER
- U7 pad 1: /TELEM_POWER_EN -> /I2C_POWER_EN
- U7 pad 4: /I2C_POWER_EN -> /TELEM_POWER_EN
- U9 pad 2: /USB2_POWER_EN -> /USB3_POWER_EN
- U9 pad 3: /USB3_POWER_EN -> /USB2_POWER_EN
- U9 pad 5: /USB3_POWER -> /USB2_POWER
- U9 pad 8: /USB2_POWER -> /USB3_POWER
Routing:
- net GND: track 13.4 -> 251.7 mm, vias 1 -> 42
- net +3V3: track 5.57 -> 165.1 mm, vias 0 -> 11
- net +5V_NANOPI: track 0.00 -> 126.6 mm, vias 0 -> 1
- net /V_peripheral: track 21.3 -> 120.7 mm, vias 0 -> 8
- net /LL_CTRL_POWER: track 5.06 -> 71.7 mm, vias 0 -> 4
- net +5V: track 3.47 -> 67.3 mm, vias 0 -> 1
- net /3V3_SENS: track 19.6 -> 68.0 mm, vias 0 -> 8
- net /NANOPI_POWER_EN: track 35.2 -> 81.7 mm, vias 0 -> 4
- net /GPS_POWER: track 0.00 -> 42.8 mm, vias 0 -> 4
- net Net-(R47-Pad2): track 0.00 -> 41.2 mm
- net /I2C_POWER: track 4.46 -> 45.5 mm, vias 1 -> 4
- net Net-(R48-Pad2): track 0.00 -> 40.3 mm
- net Net-(R45-Pad2): track 0.00 -> 38.6 mm
- net /RESET_CTRL_EN: track 1.40 -> 37.3 mm, vias 0 -> 4
- net /GPS_POWER_EN: track 33.5 -> 67.3 mm, vias 0 -> 6
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- added copper zone on In2.Cu, net /3V3_SENS

Commit message: nanopilot fabrication final version
Parts:
- added G***: LOGO, footprints:dog, B.Cu at (74.5, 46.0)
- added G***: LOGO, footprints:cat, B.Cu at (78.7, 46.3)
- U18: value H3LIS331DL -> VAL**
- moved REF** 12.3 mm to (102.0, 59.3)
- moved TP8 1.96 mm to (109.0, 33.0)
- moved TP4 1.95 mm to (104.9, 32.9)
- moved TP6 1.74 mm to (107.0, 32.7)
- moved R19 1.55 mm to (111.1, 32.8), turned to 0 degrees
- moved L1 1.55 mm to (90.2, 40.5)
- moved TP5 1.36 mm to (105.9, 32.1)
- moved R14 1.18 mm to (100.9, 38.6)
- moved D1 1.17 mm to (97.2, 31.9), turned to 180 degrees
- moved TP7 1.16 mm to (108.1, 32.1)
- moved D4 1.15 mm to (100.3, 31.9)
- moved D3 1.12 mm to (103.3, 31.9)
- moved D2 1.11 mm to (94.3, 31.9), turned to 0 degrees
- moved C37 1.06 mm to (93.8, 39.9), turned to 90 degrees
- moved R22 0.96 mm to (107.4, 34.9)
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Connections:
- D2 pad 2: +5V -> /LL_CTRL_POWER
- D3 pad 2: /V_peripheral -> /LL_CTRL_POWER
Routing:
- net /LL_CTRL_POWER: track 71.7 -> 134.4 mm, vias 4 -> 8
- net Net-(D1-Pad1): track 0.00 -> 35.9 mm, vias 0 -> 2
- net +3V3_NANOPI: track 11.2 -> 37.6 mm, vias 2 -> 3
- net GND: track 251.7 -> 270.8 mm, vias 42 -> 50
- net /V_peripheral: track 120.7 -> 103.3 mm
- net /TELEM_POWER: track 7.89 -> 20.6 mm
- net Net-(D2-Pad1): track 20.9 -> 27.6 mm, vias 1 -> 4
- net /V_SERVO: track 62.2 -> 67.6 mm, vias 11 -> 14
- net Net-(TP6-Pad1): track 10.8 -> 6.21 mm
- net /NANOPI_I2C_SDA: track 25.5 -> 21.6 mm
- net Net-(TP8-Pad1): track 10.6 -> 7.10 mm
- net /USB3_D+: track 16.6 -> 19.6 mm
- net Net-(TP5-Pad1): track 8.55 -> 6.20 mm
- net /STM_CTRL_BOOTLOADER: track 9.56 -> 11.6 mm
- net /5V_in: track 26.0 -> 27.9 mm
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- added copper zone on B.Cu, net GND
- added copper zone on F.Cu, net GND
- added copper zone on In2.Cu, net GND
