File: nanopilot/sensors.sch (KiCad schematic (older format))
At the start: 22 parts

Commit message: nanopi footprints and schematics footprints
Parts:
- gave numbers to parts that had none: 22
Connections:
- net labels removed: LSM_CLK, MPU_CLK
- no-connect marks 5 -> 7

Commit message: version ready to be routed
Parts:
- C36, C41: footprint Capacitors_SMD:C_0603 -> Capacitor_SMD:C_0603_1608Metric
- C37, C38, C39, C40, C43, C44, C45, C46, C47: footprint (none) -> Capacitor_SMD:C_0603_1608Metric
- C42: footprint (none) -> Capacitor_SMD:C_0603_1608Metric; symbol Device:CP -> Device:C_Small
- R33, R34, R35, R36: footprint (none) -> Resistor_SMD:R_0603_1608Metric
- U13: footprint (none) -> footprints:PQFN50P300X250X86-14N
- U14: footprint (none) -> footprints:MPU-9250_QFN-24_0.4mm
- U15: footprint (none) -> Package_SO:SOIC-8_3.9x4.9mm_P1.27mm
- U16: footprint (none) -> footprints:MS5611-01BA
- U17: footprint (none) -> footprints:LGA12R50P4X4_200X200X100
- U18: footprint (none) -> footprints:H3LIS331DL
Connections:
- net labels removed: +3V3
- wire segments 176 -> 177
Changed lines of the file:
@@
 F 0 "C41" H 1510 2070 50  0000 L CNN
 F 1 "0.1uF" H 1510 1920 50  0000 L CNN
-F 2 "Capacitors_SMD:C_0603" H 1500 2000 50  0001 C CNN
+F 2 "Capacitor_SMD:C_0603_1608Metric" H 1500 2000 50  0001 C CNN
 F 3 "https://www.murata.com/~/media/webrenewal/support/library/catalog/products/capacitor/mlcc/c03e.ashx" H 1500 2000 50  0001 C CNN
 F 4 "490-5798-1-ND" H 1500 2000 60  0001 C CNN "Digikey"
@@
 F 0 "C36" H 760 1820 50  0000 L CNN
 F 1 "10nF" H 760 1670 50  0000 L CNN
-F 2 "Capacitors_SMD:C_0603" H 750 1750 50  0001 C CNN
+F 2 "Capacitor_SMD:C_0603_1608Metric" H 750 1750 50  0001 C CNN
 F 3 "" H 750 1750 50  0001 C CNN
 F 4 "490-5771-1-ND" H 750 1750 60  0001 C CNN "Digikey"
@@
 F 0 "C38" H 1110 1820 50  0000 L CNN
 F 1 "100nF" H 1110 1670 50  0000 L CNN
-F 2 "" H 1100 1750 50  0001 C CNN
+F 2 "Capacitor_SMD:C_0603_1608Metric" H 1100 1750 50  0001 C CNN
 F 3 "" H 1100 1750 50  0001 C CNN
 F 4 "490-5798-1-ND" H 1100 1750 60  0001 C CNN "Digikey"
@@
 F 0 "C40" H 1375 3800 50  0000 L CNN
 F 1 "0.1uF" H 1375 3600 50  0000 L CNN
-F 2 "" H 1388 3550 50  0001 C CNN
+F 2 "Capacitor_SMD:C_0603_1608Metric" H 1388 3550 50  0001 C CNN
 F 3 "" H 1350 3700 50  0001 C CNN
 F 4 "490-5798-1-ND" H 1350 3700 60  0001 C CNN "Digikey"
@@
 F 0 "C37" H 825 4200 50  0000 L CNN
 F 1 "0.1uF" H 825 4000 50  0000 L CNN
-F 2 "" H 838 3950 50  0001 C CNN
+F 2 "Capacitor_SMD:C_0603_1608Metric" H 838 3950 50  0001 C CNN
 F 3 "" H 800 4100 50  0001 C CNN
 F 4 "490-5798-1-ND" H 800 4100 60  0001 C CNN "Digikey"
@@
 F 0 "U18" H 7100 5150 60  0000 C CNN
 F 1 "H3LIS331DL" H 7150 6350 60  0000 C CNN
-F 2 "" H 6900 5550 60  0001 C CNN
+F 2 "footprints:H3LIS331DL" H 6900 5550 60  0001 C CNN
 F 3 "" H 6900 5550 60  0001 C CNN
 	1    6900 5550
@@
 F 0 "C45" H 5360 5370 50  0000 L CNN
 F 1 "0.1uF" H 5360 5220 50  0000 L CNN
-F 2 "" H 5350 5300 50  0001 C CNN
+F 2 "Capacitor_SMD:C_0603_1608Metric" H 5350 5300 50  0001 C CNN
 F 3 "" H 5350 5300 50  0001 C CNN
 	1    5350 5300
-	1    0    0    -1
-$EndComp
-$Comp
-L Device:CP C?
-U 1 1 5B3079BC
-P 5050 5300
-AR Path="/5B30359F/5B3079BC" Ref="C?"  Part="1"
-AR Path="/5B301CE8/5BA09AAA/5B3079BC" Ref="C?"  Part="1"
-AR Path="/5C677B39/5B3079BC" Ref="C42"  Part="1"
-F 0 "C42" H 5075 5400 50  0000 L CNN
-F 1 "10uF" H 5075 5200 50  0000 L CNN
-F 2 "" H 5088 5150 50  0001 C CNN
-F 3 "" H 5050 5300 50  0001 C CNN
-	1    5050 5300
 	1    0    0    -1
 $EndComp
@@
 	5350 5400 5350 5550
 Wire Wire Line
-	5050 5450 5050 5550
-Wire Wire Line
 	5800 4700 5800 4900
 Wire Wire Line
@@
 F 0 "U17" H 7450 1750 60  0000 C CNN
 F 1 "LIS3MDL" H 7300 2750 60  0000 C CNN
-F 2 "" H 6850 1800 60  0001 C CNN
+F 2 "footprints:LGA12R50P4X4_200X200X100" H 6850 1800 60  0001 C CNN
 F 3 "" H 6850 1800 60  0001 C CNN
 	1    6850 1800
@@
 F 0 "C47" H 5810 1570 50  0000 L CNN
 F 1 "100nF" H 5810 1420 50  0000 L CNN
-F 2 "" H 5800 1500 50  0001 C CNN
+F 2 "Capacitor_SMD:C_0603_1608Metric" H 5800 1500 50  0001 C CNN
 F 3 "" H 5800 1500 50  0001 C CNN
 	1    5800 1500
@@
 F 0 "C43" H 5210 1320 50  0000 L CNN
 F 1 "1uF" H 5210 1170 50  0000 L CNN
-F 2 "" H 5200 1250 50  0001 C CNN
+F 2 "Capacitor_SMD:C_0603_1608Metric" H 5200 1250 50  0001 C CNN
 F 3 "" H 5200 1250 50  0001 C CNN
 	1    5200 1250
@@
 F 0 "C46" H 5460 1320 50  0000 L CNN
 F 1 "100nF" H 5460 1170 50  0000 L CNN
-F 2 "" H 5450 1250 50  0001 C CNN
+F 2 "Capacitor_SMD:C_0603_1608Metric" H 5450 1250 50  0001 C CNN
 F 3 "" H 5450 1250 50  0001 C CNN
 	1    5450 1250
@@
 Wire Wire Line
 	8650 1150 8650 1200
-$Comp
-L power:+3V3 #PWR?
-U 1 1 5B30C386
-P 8650 1150
-AR Path="/5B30359F/5B30C386" Ref="#PWR?"  Part="1"
-AR Path="/5B301CE8/5BA09AAA/5B30C386" Ref="#PWR?"  Part="1"
-AR Path="/5C677B39/5B30C386" Ref="#PWR0116"  Part="1"
-F 0 "#PWR0116" H 8650 1000 50  0001 C CNN
-F 1 "+3V3" H 8650 1290 50  0000 C CNN
-F 2 "" H 8650 1150 50  0001 C CNN
-F 3 "" H 8650 1150 50  0001 C CNN
-	1    8650 1150
-	1    0    0    -1
-$EndComp
 Text Notes 6600 750  0    60   ~ 0
 Address = 001 1110b (1E)
@@
 F 0 "U14" H 2800 1050 60  0000 C CNN
 F 1 "MPU-9250" H 2050 2100 60  0000 C CNN
-F 2 "" H 2600 1150 60  0001 C CNN
+F 2 "footprints:MPU-9250_QFN-24_0.4mm" H 2600 1150 60  0001 C CNN
 F 3 "" H 2600 1150 60  0001 C CNN
 F 4 "1428-1019-1-ND" H 2450 1600 60  0001 C CNN "Digikey"
@@
 F 0 "U13" H 2400 3100 60  0000 C CNN
 F 1 "LSM6DSM" H 2300 4150 60  0000 C CNN
-F 2 "" H 2250 3750 60  0001 C CNN
+F 2 "footprints:PQFN50P300X250X86-14N" H 2250 3750 60  0001 C CNN
 F 3 "" H 2250 3750 60  0001 C CNN
 	1    2250 3750
@@
 F 0 "U16" H 6850 2950 50  0000 C CNN
 F 1 "MS5611-01BA03" H 6600 3584 50  0000 C CNN
-F 2 "" H 6500 3250 50  0001 C CNN
+F 2 "footprints:MS5611-01BA" H 6500 3250 50  0001 C CNN
 F 3 "" H 6500 3250 50  0001 C CNN
 	1    6500 3250
@@
 F 0 "U15" H 2750 6050 50  0000 C CNN
 F 1 "24LC256" H 2700 6550 50  0000 C CNN
-F 2 "" H 2500 6300 50  0001 C CNN
+F 2 "Package_SO:SOIC-8_3.9x4.9mm_P1.27mm" H 2500 6300 50  0001 C CNN
 F 3 "http://ww1.microchip.com/downloads/en/devicedoc/21203m.pdf" H 2500 6300 50  0001 C CNN
 	1    2500 6300
@@
 F 0 "C44" H 5360 3370 50  0000 L CNN
 F 1 "1uF" H 5360 3220 50  0000 L CNN
-F 2 "" H 5350 3300 50  0001 C CNN
+F 2 "Capacitor_SMD:C_0603_1608Metric" H 5350 3300 50  0001 C CNN
 F 3 "" H 5350 3300 50  0001 C CNN
 	1    5350 3300
@@
 F 0 "C39" H 1260 6320 50  0000 L CNN
 F 1 "1uF" H 1260 6170 50  0000 L CNN
-F 2 "" H 1250 6250 50  0001 C CNN
+F 2 "Capacitor_SMD:C_0603_1608Metric" H 1250 6250 50  0001 C CNN
 F 3 "" H 1250 6250 50  0001 C CNN
 	1    1250 6250
@@
 F 0 "R35" H 10109 3096 50  0000 L CNN
 F 1 "4.7k" H 10109 3005 50  0000 L CNN
-F 2 "" H 10050 3050 50  0001 C CNN
+F 2 "Resistor_SMD:R_0603_1608Metric" H 10050 3050 50  0001 C CNN
 F 3 "~" H 10050 3050 50  0001 C CNN
 	1    10050 3050
@@
 F 0 "R36" H 10109 4146 50  0000 L CNN
 F 1 "4.7k" H 10109 4055 50  0000 L CNN
-F 2 "" H 10050 4100 50  0001 C CNN
+F 2 "Resistor_SMD:R_0603_1608Metric" H 10050 4100 50  0001 C CNN
 F 3 "~" H 10050 4100 50  0001 C CNN
 	1    10050 4100
@@
 Wire Wire Line
 	5350 5050 5350 5200
-Wire Wire Line
-	5050 5150 5050 5050
 Connection ~ 5050 5050
 Wire Wire Line
@@
 F 0 "R34" H 3959 1746 50  0000 L CNN
 F 1 "10k" H 3959 1655 50  0000 L CNN
-F 2 "" H 3900 1700 50  0001 C CNN
+F 2 "Resistor_SMD:R_0603_1608Metric" H 3900 1700 50  0001 C CNN
 F 3 "~" H 3900 1700 50  0001 C CNN
 	1    3900 1700
@@
 F 0 "R33" H 3659 3896 50  0000 L CNN
 F 1 "10k" H 3659 3805 50  0000 L CNN
-F 2 "" H 3600 3850 50  0001 C CNN
+F 2 "Resistor_SMD:R_0603_1608Metric" H 3600 3850 50  0001 C CNN
 F 3 "~" H 3600 3850 50  0001 C CNN
 	1    3600 3850
@@
 NoConn ~ 7100 3350
 NoConn ~ 7700 1600
+$Comp
+L Device:C_Small C?
+U 1 1 5B3079BC
+P 5050 5300
+AR Path="/5B30359F/5B3079BC" Ref="C?"  Part="1"
+AR Path="/5B301CE8/5BA09AAA/5B3079BC" Ref="C?"  Part="1"
+AR Path="/5C677B39/5B3079BC" Ref="C42"  Part="1"
+F 0 "C42" H 5075 5400 50  0000 L CNN
+F 1 "10uF" H 5075 5200 50  0000 L CNN
+F 2 "Capacitor_SMD:C_0603_1608Metric" H 5088 5150 50  0001 C CNN
+F 3 "490-10728-1-ND" H 5050 5300 50  0001 C CNN
+	1    5050 5300
+	1    0    0    -1
+$EndComp
+Wire Wire Line
+	5050 5050 5050 5200
+Wire Wire Line
+	5050 5400 5050 5550
+Text Label 9150 1150 2    50   ~ 0
+3V3_SENS
+Wire Wire Line
+	8650 1150 9150 1150
 $EndSCHEMATC

Commit message: routing WIP
Parts:
- U15: footprint Package_SO:SOIC-8_3.9x4.9mm_P1.27mm -> Package_SO:MSOP-8_3x3mm_P0.65mm
Changed lines of the file:
@@
 F 0 "U15" H 2750 6050 50  0000 C CNN
 F 1 "24LC256" H 2700 6550 50  0000 C CNN
-F 2 "Package_SO:SOIC-8_3.9x4.9mm_P1.27mm" H 2500 6300 50  0001 C CNN
-F 3 "http://ww1.microchip.com/downloads/en/devicedoc/21203m.pdf" H 2500 6300 50  0001 C CNN
+F 2 "Package_SO:MSOP-8_3x3mm_P0.65mm" H 2500 6300 50  0001 C CNN
+F 3 "http://ww1.microchip.com/downloads/en/DeviceDoc/24AA256-24LC256-24FC256-Data-Sheet-20001203V.pdf" H 2500 6300 50  0001 C CNN
 	1    2500 6300
 	1    0    0    -1
