File: nanopilot/Nanopilot.sch (KiCad schematic (older format))
At the start: 93 parts

Commit message: schematic
Parts:
- added C? (x2): 22uF, symbol Device:C_Small
- D?: value LED -> OC 5V IN
Connections:
- wire segments 527 -> 533
Other:
- moved on the sheet: U?

Commit message: nanopi footprints and schematics footprints
Parts:
- removed J?: ARM, symbol Nanopilot-rescue:Conn_01x04
- removed J?: servo_pwm, symbol Connector_Generic:Conn_01x08
- removed J?: servo_V+, symbol Connector_Generic:Conn_01x08
- removed J?: servo_GND, symbol Connector_Generic:Conn_01x08
- added C24, C25, C26, C27: 47uF, symbol Device:C_Small
- added J12, J13: servo_pwm_left, symbol Nanopilot-rescue:Conn_01x04
- added J14: servo_V+_left, symbol Nanopilot-rescue:Conn_01x04
- added J15: servo_V+_right, symbol Nanopilot-rescue:Conn_01x04
- added J16: servo_GND_left, symbol Nanopilot-rescue:Conn_01x04
- added J17: servo_GND_right, symbol Nanopilot-rescue:Conn_01x04
- added J7: ARM, symbol Nanopilot-rescue:Conn_01x05
- C2: renamed from C?; footprint (none) -> Capacitor_SMD:C_0603_1608Metric
- D2: renamed from D?; footprint (none) -> Diode_SMD:D_0603_1608Metric
- J1, J10, J11: renamed from J?; footprint (none) -> Connector_Molex:Molex_Pico-Lock_504050-0691_1x06-1MP_P1.50mm_Horizontal
- J2, J3: renamed from J?; footprint (none) -> Connector_JST:JST_GH_SM06B-GHS-TB_1x06-1MP_P1.25mm_Horizontal
- R8: renamed from 300k; value R -> 300k
- U1: renamed from U?; footprint (none) -> Package_SO:MSOP-12-1EP_3x4mm_P0.65mm_EP1.65x2.85mm
- U10, U8, U9: renamed from U?; footprint (none) -> Package_DFN_QFN:DFN-8-1EP_2x2mm_P0.5mm_EP1.05x1.75mm
- U11, U12: renamed from U?; footprint (none) -> Package_TO_SOT_SMD:SOT-353_SC-70-5
- U2: renamed from U?; footprint (none) -> symbols_autopilot:NanoPi_Header
- U3, U6: renamed from U?; footprint (none) -> symbols_autopilot:TPS25200_WSON_6
- U4: renamed from U?; footprint (none) -> Package_TO_SOT_SMD:SOT-223
- gave numbers to parts that had none: 73
Connections:
- wire segments 533 -> 554
- no-connect marks 2 -> 42
Other:
- note added: "(3V-8.4V)"
- note added: "UART3 RX/ADC"
- note removed: "UART3 RX"

Commit message: clean up libraries
Parts:
- U2: footprint symbols_autopilot:NanoPi_Header -> footprints:NanoPi_Header
- U3, U6: footprint symbols_autopilot:TPS25200_WSON_6 -> footprints:TPS25200_WSON_6
Changed lines of the file:
@@
 F 0 "U6" H 5900 1400 60  0000 C CNN
 F 1 "TPS25200" H 5550 1400 60  0000 C CNN
-F 2 "symbols_autopilot:TPS25200_WSON_6" H 5650 1150 60  0000 C CNN
+F 2 "footprints:TPS25200_WSON_6" H 5650 1150 60  0000 C CNN
 F 3 "" H 5650 1150 60  0000 C CNN
 	1    5650 1100
@@
 F 0 "U3" H 3200 1400 60  0000 C CNN
 F 1 "TPS25200" H 2850 1400 60  0000 C CNN
-F 2 "symbols_autopilot:TPS25200_WSON_6" H 2950 1150 60  0000 C CNN
+F 2 "footprints:TPS25200_WSON_6" H 2950 1150 60  0000 C CNN
 F 3 "" H 2950 1150 60  0000 C CNN
 	1    2950 1100
@@
 F 0 "U2" H 1450 7800 60  0000 C CNN
 F 1 "NanoPi_Air_1.1" H 3050 7800 60  0000 C CNN
-F 2 "symbols_autopilot:NanoPi_Header" H 2450 6300 60  0001 C CNN
+F 2 "footprints:NanoPi_Header" H 2450 6300 60  0001 C CNN
 F 3 "" H 2450 6300 60  0001 C CNN
 	1    2350 6350

Commit message: version ready to be routed
Parts:
- removed J10, J11: Conn_01x06, Connector_Molex:Molex_Pico-Lock_504050-0691_1x06-1MP_P1.50mm_Horizontal, symbol Connector_Generic:Conn_01x06
- removed J12, J13: servo_pwm_left, symbol Nanopilot-rescue:Conn_01x04
- removed J14: servo_V+_left, symbol Nanopilot-rescue:Conn_01x04
- removed J15: servo_V+_right, symbol Nanopilot-rescue:Conn_01x04
- removed J16: servo_GND_left, symbol Nanopilot-rescue:Conn_01x04
- removed J17: servo_GND_right, symbol Nanopilot-rescue:Conn_01x04
- removed Y1: 8MHz, symbol Device:Crystal
- added J10, J16: servo left, Connector_Molex:Molex_Pico-Lock_504050-0691_1x06-1MP_P1.50mm_Horizontal, symbol Nanopilot-rescue:Conn_01x06
- added J11, J17: servo right, Connector_Molex:Molex_Pico-Lock_504050-0691_1x06-1MP_P1.50mm_Horizontal, symbol Nanopilot-rescue:Conn_01x06
- added J12, J13: Servo Right, footprints:pin_headers_smd_2x03_P2.54mm_horizontal, symbol Connector_Generic:Conn_02x03_Odd_Even
- added J14, J15: Servo Left, footprints:pin_headers_smd_2x03_P2.54mm_horizontal, symbol Connector_Generic:Conn_02x03_Odd_Even
- added MH1, MH2, MH3, MH4: MountingHole_Pad, MountingHole:MountingHole_2.2mm_M2_Pad_Via, symbol Mechanical:MountingHole_Pad
- added R37, R38, R39, R40, R41, R42, R43, R44, R45, R46, R47, R48, R49, R50, R51, R52: 200, Resistor_SMD:R_0603_1608Metric, symbol Device:R_Small
- added TP1: Time, TestPoint:TestPoint_Pad_D1.0mm, symbol Connector:TestPoint
- added TP10: MISO, TestPoint:TestPoint_Pad_D1.0mm, symbol Connector:TestPoint
- added TP11: MOSI, TestPoint:TestPoint_Pad_D1.0mm, symbol Connector:TestPoint
- added TP12: CTS, TestPoint:TestPoint_Pad_D1.0mm, symbol Connector:TestPoint
- added TP13: RTS, TestPoint:TestPoint_Pad_D1.0mm, symbol Connector:TestPoint
- added TP14: TX, TestPoint:TestPoint_Pad_D1.0mm, symbol Connector:TestPoint
- added TP15: RX, TestPoint:TestPoint_Pad_D1.0mm, symbol Connector:TestPoint
- added TP16, TP9: SCL, TestPoint:TestPoint_Pad_D1.0mm, symbol Connector:TestPoint
- added TP17: SDA, TestPoint:TestPoint_Pad_D1.0mm, symbol Connector:TestPoint
- added TP2: CS_LSM, TestPoint:TestPoint_Pad_D1.0mm, symbol Connector:TestPoint
- added TP3: CS_MPU, TestPoint:TestPoint_Pad_D1.0mm, symbol Connector:TestPoint
- added TP4, TP5, TP6, TP7, TP8: TestPoint, TestPoint:TestPoint_Pad_D1.0mm, symbol Connector:TestPoint
- added Y1: 8MHz, Crystal:Crystal_SMD_Abracon_ABM3C-4Pin_5.0x3.2mm, symbol Device:Crystal_GND24
- C1, C10, C11, C12, C13, C14, C16, C17, C18, C19, C20, C21, C22, C23, C28, C29, C3, C30, C31, C32, C33, C34, C35, C6, C7: footprint (none) -> Capacitor_SMD:C_0603_1608Metric
- C15, C8, C9: footprint (none) -> Capacitor_SMD:C_0805_2012Metric; symbol Device:CP1 -> Device:C_Small
- C24, C25, C26, C27: footprint (none) -> Capacitor_SMD:C_1206_3216Metric
- C4, C5: footprint (none) -> Capacitor_SMD:C_0805_2012Metric
- D1, D3, D4: footprint (none) -> LED_SMD:LED_0603_1608Metric
- D2: footprint Diode_SMD:D_0603_1608Metric -> LED_SMD:LED_0603_1608Metric
- J4, J5, J6: footprint (none) -> Connector_JST:JST_GH_SM04B-GHS-TB_1x04-1MP_P1.25mm_Horizontal
- J7, J9: footprint (none) -> Connector_JST:JST_GH_SM05B-GHS-TB_1x05-1MP_P1.25mm_Horizontal
- J8: footprint (none) -> Connector_Molex:Molex_PicoBlade_53261-0971_1x09-1MP_P1.25mm_Horizontal
- L1: footprint (none) -> Inductor_SMD:L_0603_1608Metric
- R1, R10, R11, R12, R13, R14, R15, R16, R17, R18, R19, R2, R20, R21, R22, R23, R24, R25, R26, R27, R28, R29, R3, R30, R31, R32, R4, R5, R6, R7, R8, R9: footprint (none) -> Resistor_SMD:R_0603_1608Metric
Connections:
- net labels added: TIME_SYNC
- wire segments 554 -> 583
- no-connect marks 42 -> 35

Commit message: routing nanopilot WIP
Changed lines of the file:
@@
 Text Label 7300 5050 0    50   ~ 0
 ~SHDN_SENS
-Text Label 7300 5250 0    60   ~ 0
+Text Label 7300 5550 0    60   ~ 0
 I2C_POWER_EN
 Text Label 7300 5150 0    60   ~ 0
@@
 Text Label 7300 5350 0    60   ~ 0
 USB2_POWER_EN
-Text Label 7300 5450 0    60   ~ 0
+Text Label 7300 5650 0    60   ~ 0
 USB3_POWER_EN
-Text Label 7300 5550 0    60   ~ 0
+Text Label 7300 5250 0    60   ~ 0
 TELEM_POWER_EN
-Text Label 7300 5650 0    60   ~ 0
+Text Label 7300 5450 0    60   ~ 0
 GPS_POWER_EN
 Wire Wire Line
@@
 Wire Wire Line
 	10100 5550 10750 5550
-Text Label 10750 7350 2    50   ~ 0
+Text Label 10750 7650 2    50   ~ 0
 SERVO5_PWM
-Text Label 10750 7450 2    50   ~ 0
+Text Label 10750 7550 2    50   ~ 0
 SERVO6_PWM
-Text Label 10750 7650 2    50   ~ 0
+Text Label 10750 7350 2    50   ~ 0
 SERVO8_PWM
-Text Label 10750 7550 2    50   ~ 0
+Text Label 10750 7450 2    50   ~ 0
 SERVO7_PWM
 Wire Wire Line
@@
 SERVO16_PWM
 Wire Wire Line
-	7800 7950 8250 7950
-Wire Wire Line
 	7800 8050 8250 8050
 Wire Wire Line
 	7800 8150 8250 8150
 Wire Wire Line
+	7800 7950 8250 7950
+Wire Wire Line
 	7800 8250 8250 8250
-Text Label 7800 7950 0    50   ~ 0
+Text Label 7800 8150 0    50   ~ 0
 H3LIS_INT
-Text Label 7800 8050 0    50   ~ 0
+Text Label 7800 8250 0    50   ~ 0
 LIS3MDL_INT
-Text Label 7800 8150 0    50   ~ 0
+Text Label 7800 7950 0    50   ~ 0
 MPU_INT
-Text Label 7800 8250 0    50   ~ 0
+Text Label 7800 8050 0    50   ~ 0
 LSM_INT1
 $Comp
@@
 P 12200 900
 AR Path="/5B301CE8/5E13DAFA" Ref="#PWR?"  Part="1"
-AR Path="/5E13DAFA" Ref="#PWR?"  Part="1"
-F 0 "#PWR?" H 12200 750 50  0001 C CNN
+AR Path="/5E13DAFA" Ref="#PWR0116"  Part="1"
+F 0 "#PWR0116" H 12200 750 50  0001 C CNN
 F 1 "+3V3" H 12215 1073 50  0000 C CNN
 F 2 "" H 12200 900 50  0001 C CNN
@@
 P 12250 2100
 AR Path="/5B301CE8/5E13DC1B" Ref="#PWR?"  Part="1"
-AR Path="/5E13DC1B" Ref="#PWR?"  Part="1"
-F 0 "#PWR?" H 12250 1950 50  0001 C CNN
+AR Path="/5E13DC1B" Ref="#PWR0131"  Part="1"
+F 0 "#PWR0131" H 12250 1950 50  0001 C CNN
 F 1 "+3V3" H 12265 2273 50  0000 C CNN
 F 2 "" H 12250 2100 50  0001 C CNN
@@
 P 12300 3350
 AR Path="/5B301CE8/5E13DD3C" Ref="#PWR?"  Part="1"
-AR Path="/5E13DD3C" Ref="#PWR?"  Part="1"
-F 0 "#PWR?" H 12300 3200 50  0001 C CNN
+AR Path="/5E13DD3C" Ref="#PWR0132"  Part="1"
+F 0 "#PWR0132" H 12300 3200 50  0001 C CNN
 F 1 "+3V3" H 12315 3523 50  0000 C CNN
 F 2 "" H 12300 3350 50  0001 C CNN

Commit message: routing WIP
Changed lines of the file:
@@
 	1    0    0    -1
 $EndComp
-Text Label 14550 3600 0    60   ~ 0
+Text Label 14500 3500 0    60   ~ 0
 I2C_POWER
 $Comp
@@
 	1    0    0    -1
 $EndComp
-Text Label 12750 3900 0    60   ~ 0
+Text Label 12750 3800 0    60   ~ 0
 I2C_POWER_EN
 $Comp
@@
 L Device:C_Small C32
 U 1 1 5B27ABB0
-P 15400 3800
-F 0 "C32" H 15410 3870 50  0000 L CNN
-F 1 "0.1uF" H 15410 3720 50  0000 L CNN
-F 2 "Capacitor_SMD:C_0603_1608Metric" H 15400 3800 50  0001 C CNN
-F 3 "" H 15400 3800 50  0001 C CNN
-	1    15400 3800
+P 15100 3800
+F 0 "C32" H 15110 3870 50  0000 L CNN
+F 1 "0.1uF" H 15110 3720 50  0000 L CNN
+F 2 "Capacitor_SMD:C_0603_1608Metric" H 15100 3800 50  0001 C CNN
+F 3 "" H 15100 3800 50  0001 C CNN
+	1    15100 3800
 	1    0    0    1
 $EndComp
@@
 L Device:C_Small C29
 U 1 1 5B27ABCA
-P 15100 3800
-F 0 "C29" H 15110 3870 50  0000 L CNN
-F 1 "0.1uF" H 15110 3720 50  0000 L CNN
-F 2 "Capacitor_SMD:C_0603_1608Metric" H 15100 3800 50  0001 C CNN
-F 3 "" H 15100 3800 50  0001 C CNN
-	1    15100 3800
+P 15400 3800
+F 0 "C29" H 15410 3870 50  0000 L CNN
+F 1 "0.1uF" H 15410 3720 50  0000 L CNN
+F 2 "Capacitor_SMD:C_0603_1608Metric" H 15400 3800 50  0001 C CNN
+F 3 "" H 15400 3800 50  0001 C CNN
+	1    15400 3800
 	1    0    0    1
 $EndComp
@@
 Text Label 12650 1450 0    60   ~ 0
 NANOPI_POWER_EN
-Text Label 14650 2350 0    60   ~ 0
+Text Label 14650 2450 0    60   ~ 0
 USB2_POWER
-Text Label 12700 2650 0    60   ~ 0
+Text Label 12750 2750 0    60   ~ 0
 USB2_POWER_EN
-Text Label 12700 2750 0    60   ~ 0
+Text Label 12750 2650 0    60   ~ 0
 USB3_POWER_EN
 Text Label 14550 1250 0    60   ~ 0
 GPS_POWER
-Text Label 14500 3500 0    60   ~ 0
+Text Label 14500 3600 0    60   ~ 0
 TELEM_POWER
-Text Label 12700 3800 0    60   ~ 0
+Text Label 12650 3900 0    60   ~ 0
 TELEM_POWER_EN
 Text Label 12700 1550 0    60   ~ 0
@@
 Text Label 7300 5050 0    50   ~ 0
 ~SHDN_SENS
-Text Label 7300 5550 0    60   ~ 0
+Text Label 7300 5250 0    60   ~ 0
 I2C_POWER_EN
 Text Label 7300 5150 0    60   ~ 0
@@
 Text Label 7300 5650 0    60   ~ 0
 USB3_POWER_EN
-Text Label 7300 5250 0    60   ~ 0
+Text Label 7300 5550 0    60   ~ 0
 TELEM_POWER_EN
 Text Label 7300 5450 0    60   ~ 0
@@
 Wire Wire Line
 	14500 2450 15250 2450
-Text Label 14650 2450 0    60   ~ 0
+Text Label 14650 2350 0    60   ~ 0
 USB3_POWER
 Wire Wire Line
@@
 L Device:R_Small R?
 U 1 1 5CF1F58D
-P 12550 3600
+P 12300 3600
 AR Path="/5B301CE8/5CF1F58D" Ref="R?"  Part="1"
 AR Path="/5CF1F58D" Ref="R29"  Part="1"
-F 0 "R29" H 12609 3646 50  0000 L CNN
-F 1 "10k" H 12609 3555 50  0000 L CNN
-F 2 "Resistor_SMD:R_0603_1608Metric" H 12550 3600 50  0001 C CNN
-F 3 "~" H 12550 3600 50  0001 C CNN
-	1    12550 3600
+F 0 "R29" H 12359 3646 50  0000 L CNN
+F 1 "10k" H 12359 3555 50  0000 L CNN
+F 2 "Resistor_SMD:R_0603_1608Metric" H 12300 3600 50  0001 C CNN
+F 3 "~" H 12300 3600 50  0001 C CNN
+	1    12300 3600
 	1    0    0    -1
 $EndComp
@@
 L Device:R_Small R?
 U 1 1 5CF1F595
-P 12300 3600
+P 12550 3600
 AR Path="/5B301CE8/5CF1F595" Ref="R?"  Part="1"
 AR Path="/5CF1F595" Ref="R26"  Part="1"
-F 0 "R26" H 12359 3646 50  0000 L CNN
-F 1 "10k" H 12359 3555 50  0000 L CNN
-F 2 "Resistor_SMD:R_0603_1608Metric" H 12300 3600 50  0001 C CNN
-F 3 "~" H 12300 3600 50  0001 C CNN
-	1    12300 3600
+F 0 "R26" H 12609 3646 50  0000 L CNN
+F 1 "10k" H 12609 3555 50  0000 L CNN
+F 2 "Resistor_SMD:R_0603_1608Metric" H 12550 3600 50  0001 C CNN
+F 3 "~" H 12550 3600 50  0001 C CNN
+	1    12550 3600
 	1    0    0    -1
 $EndComp

Commit message: nanopilot fabrication final version
Connections:
- wire segments 583 -> 584
Changed lines of the file:
@@
 Wire Wire Line
 	950  1300 1300 1300
-Wire Wire Line
-	6750 750  7050 750
 Connection ~ 6750 750
 Wire Wire Line
 	6200 950  6200 750
 Wire Wire Line
-	6550 750  6750 750
-Wire Wire Line
-	6200 750  6550 750
-Connection ~ 6550 750
-Wire Wire Line
-	6550 850  6550 750
-Wire Wire Line
-	6550 1200 6550 1150
-Wire Wire Line
-	6500 1200 6550 1200
-Wire Wire Line
 	6150 950  6200 950
 Wire Wire Line
@@
 	5150 950  4850 950
 Wire Wire Line
-	3750 800  3750 750
-Wire Wire Line
 	3750 1200 3750 1100
 Wire Wire Line
@@
 	-1   0    0    -1
 $EndComp
-Text Label 6850 750  0    60   ~ 0
+Text Label 7350 750  2    60   ~ 0
 V_peripheral
 $Comp
@@
 L Device:LED D3
 U 1 1 5B2739B5
-P 6550 1000
-F 0 "D3" H 6550 1100 50  0000 C CNN
-F 1 "OC PERIPHERAL" V 6700 1050 50  0000 C CNN
-F 2 "LED_SMD:LED_0603_1608Metric" H 6550 1000 50  0001 C CNN
-F 3 "" H 6550 1000 50  0001 C CNN
-	1    6550 1000
+P 7500 1000
+F 0 "D3" H 7500 1100 50  0000 C CNN
+F 1 "OC PERIPHERAL" V 7650 1050 50  0000 C CNN
+F 2 "LED_SMD:LED_0603_1608Metric" H 7500 1000 50  0001 C CNN
+F 3 "" H 7500 1000 50  0001 C CNN
+	1    7500 1000
 	0    -1   -1   0
 $EndComp
@@
 L power:GND #PWR047
 U 1 1 5B2739A0
-P 6750 1250
-F 0 "#PWR047" H 6750 1000 50  0001 C CNN
-F 1 "GND" H 6750 1100 50  0000 C CNN
-F 2 "" H 6750 1250 50  0001 C CNN
-F 3 "" H 6750 1250 50  0001 C CNN
-	1    6750 1250
+P 6750 1050
+F 0 "#PWR047" H 6750 800 50  0001 C CNN
+F 1 "GND" H 6750 900 50  0000 C CNN
+F 2 "" H 6750 1050 50  0001 C CNN
+F 3 "" H 6750 1050 50  0001 C CNN
+	1    6750 1050
 	1    0    0    -1
 $EndComp
@@
 L Device:C_Small C15
 U 1 1 5B273999
-P 6750 1050
-F 0 "C15" H 6775 1150 50  0000 L CNN
-F 1 "22uF" H 6775 950 50  0000 L CNN
-F 2 "Capacitor_SMD:C_0805_2012Metric" H 6750 1050 50  0001 C CNN
-F 3 "490-9952-1-ND" H 6750 1050 50  0001 C CNN
-	1    6750 1050
+P 6750 900
+F 0 "C15" H 6775 1000 50  0000 L CNN
+F 1 "22uF" H 6775 800 50  0000 L CNN
+F 2 "Capacitor_SMD:C_0805_2012Metric" H 6750 900 50  0001 C CNN
+F 3 "490-9952-1-ND" H 6750 900 50  0001 C CNN
+	1    6750 900
 	1    0    0    -1
 $EndComp
@@
 $EndComp
 $Comp
-L power:+5V #PWR022
-U 1 1 5B2717A8
-P 3750 750
-F 0 "#PWR022" H 3750 600 50  0001 C CNN
-F 1 "+5V" H 3750 890 50  0000 C CNN
-F 2 "" H 3750 750 50  0001 C CNN
-F 3 "" H 3750 750 50  0001 C CNN
-	1    3750 750
-	1    0    0    -1
-$EndComp
-$Comp
 L power:+5V #PWR026
 U 1 1 5B271535
@@
 $EndComp
 $Comp
-L power:+5V #PWR018
-U 1 1 5B1C82F3
-P 3500 750
-F 0 "#PWR018" H 3500 600 50  0001 C CNN
-F 1 "+5V" H 3500 890 50  0000 C CNN
-F 2 "" H 3500 750 50  0001 C CNN
-F 3 "" H 3500 750 50  0001 C CNN
-	1    3500 750
-	1    0    0    -1
-$EndComp
-$Comp
 L symbols:TPS25200 U3
 U 1 1 5B1C814D
@@
 	4100 1100 4100 1200
 Wire Wire Line
-	6750 1150 6750 1250
+	6750 1000 6750 1050
 Wire Wire Line
-	6750 750  6750 950
+	6750 750  6750 800
 Wire Wire Line
 	7200 4250 7500 4250
@@
 Wire Wire Line
 	12200 1050 12200 1150
+Text Label 4650 550  2    60   ~ 0
+LL_CTRL_POWER
+$Comp
+L power:+5V #PWR018
+U 1 1 5B1C82F3
+P 3500 750
+F 0 "#PWR018" H 3500 600 50  0001 C CNN
+F 1 "+5V" H 3500 890 50  0000 C CNN
+F 2 "" H 3500 750 50  0001 C CNN
+F 3 "" H 3500 750 50  0001 C CNN
+	1    3500 750
+	1    0    0    -1
+$EndComp
+Wire Wire Line
+	3750 550  4650 550
+Wire Wire Line
+	3750 550  3750 800
+Text Label 8250 750  2    60   ~ 0
+LL_CTRL_POWER
+Wire Wire Line
+	7500 1200 7500 1150
+Wire Wire Line
+	6500 1200 7500 1200
+Wire Wire Line
+	7500 850  7500 750
+Wire Wire Line
+	6200 750  6750 750
+Wire Wire Line
+	7500 750  8250 750
+Wire Wire Line
+	6750 750  7350 750
 $EndSCHEMATC

Commit message: change capacitors
Parts:
- C28, C29, C30, C31, C32, C33: value 0.1uF -> 1uF
- C8: value 22uF -> 100uF
Changed lines of the file:
@@
 P 15000 1550
 F 0 "C28" H 15010 1620 50  0000 L CNN
-F 1 "0.1uF" H 15010 1470 50  0000 L CNN
+F 1 "1uF" H 15010 1470 50  0000 L CNN
 F 2 "Capacitor_SMD:C_0603_1608Metric" H 15000 1550 50  0001 C CNN
 F 3 "" H 15000 1550 50  0001 C CNN
@@
 P 15300 1550
 F 0 "C31" H 15310 1620 50  0000 L CNN
-F 1 "0.1uF" H 15310 1470 50  0000 L CNN
+F 1 "1uF" H 15310 1470 50  0000 L CNN
 F 2 "Capacitor_SMD:C_0603_1608Metric" H 15300 1550 50  0001 C CNN
 F 3 "" H 15300 1550 50  0001 C CNN
@@
 P 15550 2750
 F 0 "C33" H 15560 2820 50  0000 L CNN
-F 1 "0.1uF" H 15560 2670 50  0000 L CNN
+F 1 "1uF" H 15560 2670 50  0000 L CNN
 F 2 "Capacitor_SMD:C_0603_1608Metric" H 15550 2750 50  0001 C CNN
 F 3 "" H 15550 2750 50  0001 C CNN
@@
 P 15250 2750
 F 0 "C30" H 15260 2820 50  0000 L CNN
-F 1 "0.1uF" H 15260 2670 50  0000 L CNN
+F 1 "1uF" H 15260 2670 50  0000 L CNN
 F 2 "Capacitor_SMD:C_0603_1608Metric" H 15250 2750 50  0001 C CNN
 F 3 "" H 15250 2750 50  0001 C CNN
@@
 P 15100 3800
 F 0 "C32" H 15110 3870 50  0000 L CNN
-F 1 "0.1uF" H 15110 3720 50  0000 L CNN
+F 1 "1uF" H 15110 3720 50  0000 L CNN
 F 2 "Capacitor_SMD:C_0603_1608Metric" H 15100 3800 50  0001 C CNN
 F 3 "" H 15100 3800 50  0001 C CNN
@@
 P 15400 3800
 F 0 "C29" H 15410 3870 50  0000 L CNN
-F 1 "0.1uF" H 15410 3720 50  0000 L CNN
+F 1 "1uF" H 15410 3720 50  0000 L CNN
 F 2 "Capacitor_SMD:C_0603_1608Metric" H 15400 3800 50  0001 C CNN
 F 3 "" H 15400 3800 50  0001 C CNN
@@
 F 1 "100uF" H 4375 900 50  0000 L CNN
 F 2 "Capacitor_SMD:C_0805_2012Metric" H 4350 1000 50  0001 C CNN
-F 3 "490-9952-1-ND" H 4350 1000 50  0001 C CNN
+F 3 "" H 4350 1000 50  0001 C CNN
 	1    4350 1000
 	1    0    0    -1
@@
 P 4100 1000
 F 0 "C8" H 4125 1100 50  0000 L CNN
-F 1 "22uF" H 4125 900 50  0000 L CNN
+F 1 "100uF" H 4125 900 50  0000 L CNN
 F 2 "Capacitor_SMD:C_0805_2012Metric" H 4100 1000 50  0001 C CNN
-F 3 "490-9952-1-ND" H 4100 1000 50  0001 C CNN
+F 3 "" H 4100 1000 50  0001 C CNN
 	1    4100 1000
 	1    0    0    -1
