File: nanopilot duo/Nanopilot.kicad_pcb (KiCad board)
At the start: 4 copper layers, 39 x 50.5 mm, 149 parts, among them J1 Conn_01x06, J10 SPI, J11 servo 1..8, J13 Conn_Coaxial, J14 servo 9..12, J2 Linux I2C, J3 ETHERNET, J4 USB1, J5 USB2, J6 ARM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

Commit message: finished routing
Parts:
- removed U10, U15: SDP32, footprints:SDP3x
- added C30: 10uF, Capacitor_SMD:C_0603_1608Metric, F.Cu at (86.2, 46.8)
- added D8: OC 5V PERIPH, LED_SMD:LED_0603_1608Metric, F.Cu at (88.7, 52.9)
- added D9: RTK, LED_SMD:LED_0603_1608Metric, F.Cu at (71.9, 29.0)
- added J12: I2C_differential, Connector_JST:JST_GH_SM06B-GHS-TB_1x06-1MP_P1.25mm_Horizontal, F.Cu at (80.3, 75.1)
- added R52: 600, Resistor_SMD:R_0603_1608Metric, F.Cu at (77.1, 69.1)
- added R53: 120, Resistor_SMD:R_1206_3216Metric, F.Cu at (79.5, 69.8)
- added R54: 600, Resistor_SMD:R_0603_1608Metric, F.Cu at (84.8, 70.9)
- added R55: 600, Resistor_SMD:R_0603_1608Metric, F.Cu at (77.0, 71.1)
- added R56: 120, Resistor_SMD:R_1206_3216Metric, F.Cu at (81.6, 69.8)
- added R57: 600, Resistor_SMD:R_0603_1608Metric, F.Cu at (84.0, 68.6)
- added R58: 1k, Resistor_SMD:R_0603_1608Metric, F.Cu at (73.2, 29.3)
- added U6: TPS25200, footprints:TPS25200_WSON_6, F.Cu at (86.2, 45.0)
- C28: value 100nF -> 0.1uF
- C32, C35, C36, R45, R46, U11: moved to F.Cu
- J2, J5: footprint Connector_JST:JST_GH_BM04B-GHS-TBT_1x04-1MP_P1.25mm_Vertical -> Connector_JST:JST_GH_SM04B-GHS-TB_1x04-1MP_P1.25mm_Horizontal
- R47: value 1.2k -> 64k 1%; moved to F.Cu
- R51: value 2.7k -> 1.5k; moved to F.Cu
- U12: value NEO-M8T -> NEO-M8P
- U9: value SDP32 -> PCA9615; footprint footprints:SDP3x -> Package_SO:TSSOP-10_3x3mm_P0.5mm; moved to B.Cu
- moved R51 37.5 mm to (88.7, 43.2), turned to 180 degrees
- moved R47 32.6 mm to (88.1, 47.4), turned to 270 degrees
- moved R45 28.5 mm to (83.0, 47.9), turned to 180 degrees
- moved C28 28.3 mm to (85.9, 43.2)
- moved R9 27.9 mm to (71.6, 76.5)
- moved U11 26.9 mm to (78.9, 48.8), turned to 0 degrees
- moved C41 26.6 mm to (75.6, 44.9)
- moved C35 25.5 mm to (76.3, 50.6), turned to 180 degrees
- moved U14 24.5 mm to (79.0, 45.0)
- moved R46 24.4 mm to (83.0, 46.7), turned to 180 degrees
- moved C36 24.3 mm to (76.0, 49.2)
- moved R6 24.2 mm to (72.3, 74.2), turned to 90 degrees
- moved C32 23.8 mm to (75.9, 47.9), turned to 180 degrees
- moved J2 23.1 mm to (70.5, 75.1), turned to 0 degrees
- moved J5 16.4 mm to (91.8, 67.0)
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Connections:
- C28 pad 1: /3V3_SENS -> +5V
- C31 pad 1: /3V3_SENS -> +3V3
- C42 pad 1: /3V3_SENS -> /5V_PERIPH
- J10 pad 1: +5V -> /5V_PERIPH
- J2 pad 1: +5V -> /5V_PERIPH
- J4 pad 1: +5V -> /5V_PERIPH
- J5 pad 1: +5V -> /5V_PERIPH
- J6 pad 1: +5V -> /5V_PERIPH
- J7 pad 1: +5V -> /5V_PERIPH
- R51 pad 2: GND -> Net-(R51-Pad2)
- U12 pad 15: (no net) -> /GPS_RTK_MODE
- U9 pad 1: GND -> +3V3
- U9 pad 10: GND -> /5V_PERIPH
- U9 pad 2: GND -> /STM_I2C_SDA
- U9 pad 3: GND -> (no net)
- U9 pad 4: (no net) -> /STM_I2C_SCL
- U9 pad 5: /I2C_SENS_SCL -> GND
- U9 pad 6: GND -> /DI2C_SCLM
- U9 pad 7: /3V3_SENS -> /DI2C_SCLP
- U9 pad 8: /I2C_SENS_SDA -> /DI2C_SDAP
- U9 pad 9: GND -> /DI2C_SDAM
Routing:
- net /5V_PERIPH: track 0.00 -> 91.6 mm, vias 0 -> 7
- net GND: track 359.5 -> 289.6 mm
- net +5V: track 106.7 -> 39.1 mm, vias 7 -> 2
- net +3V3_NANOPI: track 131.6 -> 98.5 mm
- net /STM_I2C_SDA: track 7.57 -> 35.3 mm, vias 1 -> 2
- net /NANOPI_I2C_SCL: track 11.2 -> 36.8 mm, vias 1 -> 2
- net /LIS3MDL_INT: track 19.5 -> 40.2 mm, vias 3 -> 2
- net /I2C_SENS_SCL: track 63.3 -> 42.7 mm, vias 5 -> 3
- net /STM_I2C_SCL: track 12.9 -> 32.9 mm, vias 1 -> 2
- net /SPI_CONN_S2: track 35.9 -> 16.8 mm
- net /NANOPI_I2C_SDA: track 11.6 -> 29.9 mm, vias 1 -> 2
- net /GPS_RTK_MODE: track 0.00 -> 16.5 mm, vias 0 -> 1
- net /I2C_SENS_SDA: track 53.1 -> 37.4 mm, vias 1 -> 3
- net /DI2C_SDAM: track 0.00 -> 14.4 mm, vias 0 -> 1
- net /3V3_SENS: track 84.2 -> 70.3 mm, vias 5 -> 4
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
Commit message: silkscreen & gerber
Parts:
- added G***: LOGO, footprints:cat, B.Cu at (83.2, 33.6)
- added G***: LOGO, footprints:dog, B.Cu at (78.4, 38.1)
- added REF**: axes_s, footprints:axes_s, F.Cu at (84.1, 43.4)
Other:
- board text added: "ARM"
- board text added: "DBG"
- board text added: "DI2C"
- board text added: "ETH"
- board text added: "I2C"
- board text added: "Linux I2C"
- board text added: "PWM"
- board text added: "PWR"
- board text added: "RX"
- board text added: "SPI"
- board text added: "USB"

Commit message: Nanopilot Duo: final BOM and some component value changes
Parts:
- removed G***: LOGO, footprints:cat
- removed G***: LOGO, footprints:dog
- removed REF**: axes_s, footprints:axes_s
- L1: value L_Small -> 0R
- L2, L3: value BLM15HD102SN1 -> 1k@100MHz
- R1: value 812k -> 820k
- R15: value 3.7k -> 3.6k
- R2: value 247k -> 249k
- R20: value 1.5k -> 3.6k
- R47: value 64k 1% -> 63.4k
- R49: value 0 -> 1k@100MHz
- R52, R54, R55, R57: value 600 -> 604
