File: nanopilot duo/Nanopilot.sch (KiCad schematic (older format))
At the start: 149 parts, among them J1 Conn_01x06, J10 SPI, J11 servo 1..8, J13 Conn_Coaxial, J14 servo 9..12, J2 Linux I2C, J3 ETHERNET, J4 USB1, J5 USB2, J6 ARM, J7 I2C, J8 DBG, J9 RX, Q1 DMN5L06WKDICT-ND, U1 LTC4419, U10 SDP32, U11 LIS3MDL, U12 NEO-M8P, U13 ICM-20602, U14 MS5611-01BA03, U15 SDP32, U2 NanoPi_Duo_2, U3 TPS25200, U4 LT1965-3.3, U5 LT1761-3.3, U7 STM32F722RETx, U8 24LC256, U9 SDP32, Y1 8MHz

Commit message: finished routing
Parts:
- removed R47: 1.2k, Resistor_SMD:R_0603_1608Metric, symbol Device:R_Small
- removed R51: 2.7k, Resistor_SMD:R_0603_1608Metric, symbol Device:R_Small
- removed U10, U15, U9: SDP32, footprints:SDP3x, symbol sensors:SDP32
- added C30: 10uF, Capacitor_SMD:C_0603_1608Metric, symbol Device:C_Small
- added D8: OC 5V PERIPH, LED_SMD:LED_0603_1608Metric, symbol Device:LED
- added D9: RTK, LED_SMD:LED_0603_1608Metric, symbol Device:LED
- added J12: I2C_differential, Connector_JST:JST_GH_SM06B-GHS-TB_1x06-1MP_P1.25mm_Horizontal, symbol Connector_Generic:Conn_01x06
- added R47: 64k 1%, Resistor_SMD:R_0603_1608Metric, symbol Device:R
- added R51: 1.5k, Resistor_SMD:R_0603_1608Metric, symbol Device:R
- added R52, R54, R55, R57: 600, Resistor_SMD:R_0603_1608Metric, symbol Device:R_Small
- added R53, R56: 120, Resistor_SMD:R_1206_3216Metric, symbol Device:R_Small
- added R58: 1k, Resistor_SMD:R_0603_1608Metric, symbol Device:R_Small
- added U6: TPS25200, footprints:TPS25200_WSON_6, symbol symbols:TPS25200
- added U9: PCA9615, Package_SO:TSSOP-10_3x3mm_P0.5mm, symbol symbols:PCA9615
- C28: value 100nF -> 0.1uF
- J2, J5: footprint Connector_JST:JST_GH_BM04B-GHS-TBT_1x04-1MP_P1.25mm_Vertical -> Connector_JST:JST_GH_SM04B-GHS-TB_1x04-1MP_P1.25mm_Horizontal
Connections:
- net +3V3: now also C31.1, U9.1 (VDDA)
- net +5V: now also C28.1, U6.4 (EN), U6.6 (IN); no longer J10.1 (Pin_1), J2.1 (Pin_1), J4.1 (Pin_1), J5.1 (Pin_1), J6.1 (Pin_1), J7.1 (Pin_1)
- net 3V3_SENS: no longer C28.1, C31.1, C42.1
- net GND: now also C30.2, J12.6 (Pin_6), R47.2, R54.2, R57.2, R58.2, U6.5 (GND), U6.7 (GNDPAD), U9.5 (VSS)
- net LL_CTRL_POWER: now also D8.2 (A)
- net STM_I2C_SCL: now also U9.4 (SCL)
- net STM_I2C_SDA: now also U9.2 (SDA)
- net GPS_RTK_MODE: now reaches U12.15 (EXTINT1)
- net GPS_RTK_MODE: now also D9.2 (A)
- new net: R47.1, U6.2 (ILIM)
- new net: R51.2, U6.3 (~FAULT)
- new net: D8.1 (K), R51.1
- new net: D9.1 (K), R58.1
- new net 5V_PERIPH: C30.1, C42.1, J10.1 (Pin_1), J12.1 (Pin_1), J2.1 (Pin_1), J4.1 (Pin_1), J5.1 (Pin_1), J6.1 (Pin_1), J7.1 (Pin_1), R52.1, R55.1, U6.1 (OUT), U9.10 (VDDB)
- new net DI2C_SCLM: J12.3 (Pin_3), R53.2, R54.1, U9.6 (DSCLM)
- new net DI2C_SCLP: J12.2 (Pin_2), R52.2, R53.1, U9.7 (DSCLP)
- new net DI2C_SDAM: J12.5 (Pin_5), R56.2, R57.1, U9.9 (DSDAM)
- new net DI2C_SDAP: J12.4 (Pin_4), R55.2, R56.1, U9.8 (DSDAP)
- no-connect marks 22 -> 19
Other:
- note added: "1.5 A limit"
- note removed: "SDP3x I2C addr\n0k 0x21\n1.2k 0x22\n2.7k 0x23"
- note removed: "Sensor options:\nSDP32 (125Pa) up to 50km/h\nSDP31 (500Pa) up to 100km/h\nSDP33 (1500Pa) up to 180km/h"
- note removed: "differential pressure:\nangle of attack"
- note removed: "differential pressure:\nangle of sideslip"
- note removed: "differential pressure:\ndynamic pressure"
- moved on the sheet: BT1, C15, C16, C29, C32, C33, C34, C35, C36, C37, C38, C39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

Commit message: Nanopilot Duo: final BOM and some component value changes
Parts:
- L1: value L_Small -> 0R
- L2, L3: value BLM15HD102SN1 -> 1k@100MHz; digikey (none) -> 445-8672-1-ND
- R1: value 812k -> 820k
- R15: value 3.7k -> 3.6k
- R2: value 247k -> 249k
- R20: value 1.5k -> 3.6k
- R47: value 64k 1% -> 63.4k
- R49: value 0 -> 1k@100MHz
- R52, R54, R55, R57: value 600 -> 604
Other:
- note added: "3.6V(3V)..8.4V"
- note added: "V1<4.5V"
- note added: "V2 used if V1 < 3.5V"
- note removed: "(3V-8.4V)"
Changed lines of the file:
@@
 P 900 2550
 F 0 "R1" H 930 2570 50  0000 L CNN
-F 1 "812k" V 800 2500 50  0000 L CNN
+F 1 "820k" V 800 2500 50  0000 L CNN
 F 2 "Resistor_SMD:R_0603_1608Metric" H 900 2550 50  0001 C CNN
 F 3 "" H 900 2550 50  0001 C CNN
@@
 P 900 2850
 F 0 "R2" H 930 2870 50  0000 L CNN
-F 1 "247k" V 800 2750 50  0000 L CNN
+F 1 "249k" V 800 2750 50  0000 L CNN
 F 2 "Resistor_SMD:R_0603_1608Metric" H 900 2850 50  0001 C CNN
 F 3 "" H 900 2850 50  0001 C CNN
@@
 P 2950 3000
 F 0 "R15" V 3030 3000 50  0000 C CNN
-F 1 "3.7k" V 2950 3000 50  0000 C CNN
+F 1 "3.6k" V 2950 3000 50  0000 C CNN
 F 2 "Resistor_SMD:R_0603_1608Metric" V 2880 3000 50  0001 C CNN
 F 3 "" H 2950 3000 50  0001 C CNN
@@
 P 3600 1200
 F 0 "R20" V 3680 1200 50  0000 C CNN
-F 1 "1.5k" V 3600 1200 50  0000 C CNN
+F 1 "3.6k" V 3600 1200 50  0000 C CNN
 F 2 "Resistor_SMD:R_0603_1608Metric" V 3530 1200 50  0001 C CNN
 F 3 "" H 3600 1200 50  0001 C CNN
@@
 P 12300 7050
 F 0 "L2" V 12122 7050 50  0000 C CNN
-F 1 "BLM15HD102SN1" V 12213 7050 50  0000 C CNN
+F 1 "1k@100MHz" V 12213 7050 50  0000 C CNN
 F 2 "Inductor_SMD:L_0603_1608Metric" H 12300 7050 50  0001 C CNN
 F 3 "~" H 12300 7050 50  0001 C CNN
+F 4 "445-8672-1-ND" V 12300 7050 50  0001 C CNN "digikey"
 	1    12300 7050
 	0    1    1    0
@@
 P 12300 7150
 F 0 "L3" V 12122 7150 50  0000 C CNN
-F 1 "BLM15HD102SN1" V 12213 7150 50  0000 C CNN
+F 1 "1k@100MHz" V 12213 7150 50  0000 C CNN
 F 2 "Inductor_SMD:L_0603_1608Metric" H 12300 7150 50  0001 C CNN
 F 3 "~" H 12300 7150 50  0001 C CNN
+F 4 "445-8672-1-ND" V 12300 7150 50  0001 C CNN "digikey"
 	1    12300 7150
 	0    1    1    0
@@
 P 14550 7150
 F 0 "R49" V 14500 7100 50  0000 C CNN
-F 1 "0" V 14445 7150 50  0000 C CNN
+F 1 "1k@100MHz" V 14550 7150 50  0000 C CNN
 F 2 "Resistor_SMD:R_0603_1608Metric" H 14550 7150 50  0001 C CNN
 F 3 "~" H 14550 7150 50  0001 C CNN
@@
 AR Path="/60021BFF" Ref="L1"  Part="1"
 F 0 "L1" H 12047 7396 50  0000 L CNN
-F 1 "L_Small" V 11950 7300 50  0000 L CNN
+F 1 "0R" V 11950 7300 50  0000 L CNN
 F 2 "Inductor_SMD:L_0603_1608Metric" H 12000 7350 50  0001 C CNN
 F 3 "~" H 12000 7350 50  0001 C CNN
@@
 SERVO10_PWM
 Text Notes 1050 3350 0    50   ~ 0
-(3V-8.4V)
+3.6V(3V)..8.4V
 Wire Wire Line
 	1150 1000 1150 900
@@
 P 7900 1500
 F 0 "R47" V 7980 1500 50  0000 C CNN
-F 1 "64k 1%" V 7800 1500 50  0000 C CNN
+F 1 "63.4k" V 7800 1500 50  0000 C CNN
 F 2 "Resistor_SMD:R_0603_1608Metric" V 7830 1500 50  0001 C CNN
 F 3 "" H 7900 1500 50  0001 C CNN
@@
 P 15700 9150
 F 0 "R55" H 15759 9196 50  0000 L CNN
-F 1 "600" H 15759 9105 50  0000 L CNN
+F 1 "604" H 15759 9105 50  0000 L CNN
 F 2 "Resistor_SMD:R_0603_1608Metric" H 15700 9150 50  0001 C CNN
 F 3 "~" H 15700 9150 50  0001 C CNN
@@
 P 15700 9550
 F 0 "R57" H 15759 9596 50  0000 L CNN
-F 1 "600" H 15759 9505 50  0000 L CNN
+F 1 "604" H 15759 9505 50  0000 L CNN
 F 2 "Resistor_SMD:R_0603_1608Metric" H 15700 9550 50  0001 C CNN
 F 3 "~" H 15700 9550 50  0001 C CNN
@@
 P 14850 9150
 F 0 "R52" H 14909 9196 50  0000 L CNN
-F 1 "600" H 14909 9105 50  0000 L CNN
+F 1 "604" H 14909 9105 50  0000 L CNN
 F 2 "Resistor_SMD:R_0603_1608Metric" H 14850 9150 50  0001 C CNN
 F 3 "~" H 14850 9150 50  0001 C CNN
@@
 P 14850 9550
 F 0 "R54" H 14909 9596 50  0000 L CNN
-F 1 "600" H 14909 9505 50  0000 L CNN
+F 1 "604" H 14909 9505 50  0000 L CNN
 F 2 "Resistor_SMD:R_0603_1608Metric" H 14850 9550 50  0001 C CNN
 F 3 "~" H 14850 9550 50  0001 C CNN
@@
 Wire Wire Line
 	5050 4800 5050 4850
+Text Notes 3000 3200 0    50   ~ 0
+V1<4.5V
+Text Notes 2350 3550 0    50   ~ 0
+V2 used if V1 < 3.5V
 $EndSCHEMATC
