File: power-supply/power-supply.sch (KiCad schematic (older format))
At the start: 70 parts

Commit message: airdata & power supply pcb
Parts:
- removed C?: 10uF, symbol Device:C_Small
- removed C?: 220uF 16V, symbol Device:CP_Small
- removed J?: switch, symbol Connector_Generic:Conn_01x02
- removed Q?: Q_PMOS_DGS, symbol Device:Q_PMOS_DGS
- added C11: 10uF, Capacitor_SMD:C_0603_1608Metric, symbol Device:C_Small
- added C21, C27, C28, C29, C30, C31, C32, C33, C34, C35: 47uF 10V, Capacitor_SMD:C_0805_2012Metric, symbol Device:C_Small
- added J10: Power_solder, Connector_PinHeader_2.00mm:PinHeader_1x06_P2.00mm_Vertical, symbol Connector_Generic:Conn_01x06
- added J6: switch, Connector_Molex:Molex_PicoBlade_53047-0610_1x03_P1.25mm_Vertical, symbol Connector_Generic:Conn_01x03
- added J8: BATT_B_solder, Connector_PinHeader_2.00mm:PinHeader_1x02_P2.00mm_Vertical, symbol Connector_Generic:Conn_01x02
- added J9: BATT_A_solder, Connector_PinHeader_2.00mm:PinHeader_1x02_P2.00mm_Vertical, symbol Connector_Generic:Conn_01x02
- added MH1, MH2: MountingHole_Pad, MountingHole:MountingHole_2.2mm_M2_Pad_Via, symbol Mechanical:MountingHole_Pad
- added Q1: Q_PMOS_GSD, Package_TO_SOT_SMD:SOT-323_SC-70, symbol Device:Q_PMOS_GSD
- C1, C10, C12, C13, C15, C16, C17, C18, C19, C2, C4, C6, C9: renamed from C?; footprint (none) -> Capacitor_SMD:C_0603_1608Metric
- C14: renamed from C?; value 0.1uF -> 1uF; footprint (none) -> Capacitor_SMD:C_0603_1608Metric
- C20, C22, C23, C24: renamed from C?; footprint (none) -> Capacitor_SMD:C_0805_2012Metric; part (none) -> GRM21BR61C226ME44L
- C25, C26: renamed from C?; footprint (none) -> Capacitor_Tantalum_SMD:CP_EIA-7343-31_Kemet-D
- C3: renamed from C?; footprint (none) -> Capacitor_SMD:C_0603_1608Metric; part (none) -> C1608X5R1A106K080AC
- C5, C7, C8: renamed from C?; footprint (none) -> Capacitor_SMD:C_0805_2012Metric
- D1, D2, D3, D4: renamed from D?; footprint (none) -> LED_SMD:LED_0603_1608Metric
- J1, J5: renamed from J?; footprint (none) -> Connector_PinHeader_2.00mm:PinHeader_1x02_P2.00mm_Vertical
- J2: renamed from J?; footprint (none) -> footprints:USB_Micro-B_Molex-105133-0001_or_105017-0001; part (none) -> molex-105017-0001
- J3, J4: renamed from J?; footprint (none) -> Connector_JST:JST_PH_S2B-PH-SM4-TB_1x02-1MP_P2.00mm_Horizontal
- J7: renamed from J?; footprint (none) -> Connector_Molex:Molex_Pico-Lock_504050-0691_1x06-1MP_P1.50mm_Horizontal
- JP1, JP2, JP3: renamed from JP?; footprint (none) -> Jumper:SolderJumper-2_P1.3mm_Open_TrianglePad1.0x1.5mm
- L1, L2: renamed from L?; footprint (none) -> footprints:L-TDK-SPM6530
- R1, R10, R11, R12, R13, R14, R15, R16, R17, R18, R19, R2, R20, R21, R22, R23, R4, R6, R7, R8, R9: renamed from R?; footprint (none) -> Resistor_SMD:R_0603_1608Metric
- R3: renamed from R?; footprint (none) -> Resistor_SMD:R_2512_6332Metric; part (none) -> WSL2512R0200FEA18
- R5: renamed from R?; value 220k -> 1M; footprint (none) -> Resistor_SMD:R_0603_1608Metric
- U1: renamed from U?; footprint (none) -> Package_TO_SOT_SMD:SOT-23-5
- U2: renamed from U?; footprint (none) -> Package_DFN_QFN:DFN-10-1EP_3x3mm_P0.5mm_EP1.55x2.48mm
- U3: renamed from U?; footprint (none) -> footprints:VQFN-20-4.5x3.5
- gave numbers to parts that had none: 1
Connections:
- wire segments 276 -> 327

Commit message: power supply notes
Other:
- note added: "should be 200k"
Changed lines of the file:
@@
 Wire Wire Line
 	3150 4100 3600 4100
+Text Notes 2650 1200 0    50   ~ 0
+should be 200k
+Text Notes 7400 1600 0    50   ~ 0
+should be 200k
 $EndSCHEMATC
